File: rjx_training_kit/peripherals.kicad_sch (KiCad schematic)
At the start: 12 parts, among them J3 USB_OTG, SW3 SW_Push, U2 BME280, U3 DS3231M, U4 LTC-4627JD, U5 LIS3DH, U7 EMIF02-USB03F2

Commit message: Update
Parts:
- added BT1: 3V, symbol Device:Battery_Cell
- added C3: 0.1uF, symbol Device:C
- added C4, C5, C6: 100nF, symbol Device:C
- added C7: 10uF, symbol Device:C
- added Q1: BC847, Package_TO_SOT_SMD:SOT-23, symbol Transistor_BJT:BC847
- added R10, R9: 4.7k, symbol Device:R_US
- added R11, R6: 10k, symbol Device:R_US
- added R12: R, symbol Device:R_US
- added R7: 1k, symbol Device:R_US
- added R8: 240, symbol Device:R_US
- D2: value LED -> User LED (Green)
- RV1: value R_Potentiometer_Trim_US -> 10k
- RV2: value R_Potentiometer_US -> 10k
Connections:
- net GND: now reaches RV1.1
- net GND: now also D2.1 (K), DS1.1 (VSS), DS1.5 (R/W), RV2.1, SW3.1, U2.1 (GND), U2.5 (SDO), U2.7 (GND), U3.10 (GND), U3.11 (GND), U3.12 (GND), U3.13 (GND), U3.5 (GND), U3.6 (GND), U3.7 (GND), U3.8 (GND), U3.9 (GND), U5.10 (GND), U5.12 (GND), U5.13 (ADC3), U5.15 (ADC2), U5.16 (ADC1), U5.5 (GND), BT1.2 (-), C3.2, C4.2, C5.2, C6.2, C7.2, Q1.2 (E), R6.2
- net at RV1.2: now also DS1.3 (VO)
- net +5V: now reaches RV1.3
- net +5V: now also DS1.2 (VDD), R8.2
- net at DS1.15 (LED(+)): now also R8.1
- net at DS1.16 (LED(-)): now also Q1.3 (C)
- net at U3.1 (32KHZ): now also R10.2
- net at U3.14 (VBAT): now also BT1.1 (+)
- net +3.3V: now reaches U3.2 (VCC)
- net +3.3V: now also RV2.3, C3.1, R10.1, R11.1, R9.1
- net at U3.3 (~{INT}/SQW): now also R9.2
- net at D2.2 (A): now also R12.2
- net +3V3: now reaches U5.1 (VDD_IO)
- net +3V3: now also U2.2 (CSB), U2.6 (VDDIO), U2.8 (VDD), U5.14 (VDD), C4.1, C5.1, C6.1, C7.1
- net at SW3.2: now also R11.2
- new net: Q1.1 (B), R7.2
- new net: R6.1, R7.1
- no-connect marks 0 -> 1
Other:
- note added: "Accelerometer"
- note added: "I2C Address: 0x68"
- note added: "I2C Address: 0x76"
- note added: "LCD"
- note added: "Potentiometer"
- note added: "RTC"
- note added: "Temperature & Humidity Sensor"
- note added: "User Button"
- note added: "User LED"
- moved on the sheet: BZ1, D2, DS1, J3, RV1, RV2, SW3, U2, U3, U4, U5, U7

Commit message: Update
Parts:
- removed DS1: WC1602A, Display:WC1602A, symbol Display_Character:WC1602A
- removed J3: USB_OTG, symbol Connector:USB_OTG
- removed Q1: BC847, Package_TO_SOT_SMD:SOT-23, symbol Transistor_BJT:BC847
- removed R10, R9: 4.7k, symbol Device:R_US
- removed R6: 10k, symbol Device:R_US
- removed R7: 1k, symbol Device:R_US
- removed R8: 240, symbol Device:R_US
- removed RV1: 10k, symbol Device:R_Potentiometer_Trim_US
- removed U4: LTC-4627JD, Display_7Segment:LTC-4627Jx, symbol Display_Character:LTC-4627JD
- removed U7: EMIF02-USB03F2, FLIP-CHIP11_1P44X1P94_STM, symbol emif02-usb03f2:EMIF02-USB03F2
- added Q7: BC847, Package_TO_SOT_SMD:SOT-23, symbol Transistor_BJT:BC847
- added R26, R27: 4.7k, symbol Device:R_US
- R12: value R -> 470
Connections:
- net +3.3V: now also Q7.3 (C)
- net +3V3: now also R26.1, R27.1
- net GND: now also BZ1.2 (-)
- net PC4: now reaches R12.1
- net PB11: now reaches U3.15 (SDA)
- net PB11: now also U2.3 (SDI), R27.2
- net PB10: now reaches U3.16 (SCL)
- net PB10: now also U2.4 (SCK), R26.2
- net at BZ1.1 (+): now also Q7.2 (E)
- net PC5: now reaches R11.2, SW3.2
- net PA1: now reaches RV2.2
- new net PE7: Q7.1 (B)
- no-connect marks 1 -> 3
Other:
- note added: "ADC1_IN1"
- note added: "Buzzer"
- note added: "I2C Pullups"
- note added: "I2C2_SCL"
- note added: "I2C2_SDA"
- note removed: "LCD"
- moved on the sheet: BT1, BZ1, C3, C4, C5, C6, C7, D2, R11, R12, RV2, SW3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

Commit message: Update
Connections:
- net +3.3V is gone; now on net +3V3: C3.1, Q7.3 (C), R11.1, RV2.3, U3.2 (VCC)
- net PE0: now reaches U5.11 (INT1)
- net PA5: now reaches U5.4 (SPC)
- net PA7: now reaches U5.6 (SDI)
- net PA6: now reaches U5.7 (SDO)
- net PE2: now reaches U5.8 (CS)
- net PE1: now reaches U5.9 (INT2)
Other:
- note added: "LIS3DH_INT1"
- note added: "LIS3DH_INT2"
- note added: "SPI1_MISO"
- note added: "SPI1_MOSI"
- note added: "SPI1_SCK"
- note added: "SPI_CS"
Changed lines of the file:
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@@
 	(wire
 		(pts
-			(xy 147.32 49.53) (xy 158.75 49.53)
+			(xy 151.13 49.53) (xy 158.75 49.53)
 		)
 		(stroke
@@
 	(wire
 		(pts
-			(xy 147.32 57.15) (xy 158.75 57.15)
+			(xy 151.13 57.15) (xy 158.75 57.15)
 		)
 		(stroke
@@
 	(wire
 		(pts
-			(xy 147.32 62.23) (xy 158.75 62.23)
+			(xy 151.13 62.23) (xy 158.75 62.23)
 		)
 		(stroke
@@
 	(wire
 		(pts
-			(xy 147.32 54.61) (xy 158.75 54.61)
+			(xy 151.13 54.61) (xy 158.75 54.61)
 		)
 		(stroke
@@
 	(wire
 		(pts
-			(xy 147.32 52.07) (xy 158.75 52.07)
+			(xy 151.13 52.07) (xy 158.75 52.07)
 		)
 		(stroke
@@
 	(wire
 		(pts
-			(xy 147.32 59.69) (xy 158.75 59.69)
+			(xy 151.13 59.69) (xy 158.75 59.69)
 		)
 		(stroke
@@
 		)
 	)
+	(text "SPI1_MISO"
+		(exclude_from_sim no)
+		(at 137.922 54.864 0)
+		(effects
+			(font
+				(size 1.27 1.27)
+			)
+		)
+	)
 	(text "RTC"
 		(exclude_from_sim no)
@@
 		)
 	)
+	(text "SPI1_SCK"
+		(exclude_from_sim no)
+		(at 137.414 59.69 0)
+		(effects
+			(font
+				(size 1.27 1.27)
+			)
+		)
+	)
 	(text "User Button"
 		(exclude_from_sim no)
@@
 		)
 	)
+	(text "LIS3DH_INT1"
+		(exclude_from_sim no)
+		(at 138.938 49.784 0)
+		(effects
+			(font
+				(size 1.27 1.27)
+			)
+		)
+	)
 	(text "I2C Address: 0x76"
 		(exclude_from_sim no)
@@
 		)
 	)
+	(text "SPI1_MOSI"
+		(exclude_from_sim no)
+		(at 137.922 57.404 0)
+		(effects
+			(font
+				(size 1.27 1.27)
+			)
+		)
+	)
+	(text "SPI_CS"
+		(exclude_from_sim no)
+		(at 136.144 61.976 0)
+		(effects
+			(font
+				(size 1.27 1.27)
+			)
+		)
+	)
 	(text "I2C Address: 0x68"
 		(exclude_from_sim no)
@@
 		)
 	)
+	(text "LIS3DH_INT2"
+		(exclude_from_sim no)
+		(at 138.938 52.324 0)
+		(effects
+			(font
+				(size 1.27 1.27)
+			)
+		)
+	)
 	(label "PC5"
 		(at 257.81 39.37 0)
@@
 		)
 	)
+	(label "PA5"
+		(at 157.48 59.69 180)
+		(fields_autoplaced yes)
+		(effects
+			(font
+				(size 1.27 1.27)
+			)
+			(justify right bottom)
+		)
+	)
+	(label "PA7"
+		(at 157.48 57.15 180)
+		(fields_autoplaced yes)
+		(effects
+			(font
+				(size 1.27 1.27)
+			)
+			(justify right bottom)
+		)
+	)
 	(label "PB11"
 		(at 80.01 107.95 180)
@@
 		)
 	)
+	(label "PE1"
+		(at 157.48 52.07 180)
+		(fields_autoplaced yes)
+		(effects
+			(font
+				(size 1.27 1.27)
+			)
+			(justify right bottom)
+		)
+	)
+	(label "PE2"
+		(at 153.67 62.23 0)
+		(fields_autoplaced yes)
+		(effects
+			(font
+				(size 1.27 1.27)
+			)
+			(justify left bottom)
+		)
+	)
 	(label "PA1"
 		(at 260.35 144.78 0)
@@
 		)
 	)
+	(label "PA6"
+		(at 157.48 54.61 180)
+		(fields_autoplaced yes)
+		(effects
+			(font
+				(size 1.27 1.27)
+			)
+			(justify right bottom)
+		)
+	)
 	(label "PB10"
 		(at 52.07 107.95 180)
@@
 		)
 	)
+	(label "PE0"
+		(at 157.48 49.53 180)
+		(fields_autoplaced yes)
+		(effects
+			(font
+				(size 1.27 1.27)
+			)
+			(justify right bottom)
+		)
+	)
 	(label "PB11"
 		(at 83.82 171.45 0)
@@
 		)
 	)
+	(hierarchical_label "PA5"
+		(shape input)
+		(at 151.13 59.69 180)
+		(fields_autoplaced yes)
+		(effects
+			(font
+				(size 1.27 1.27)
+			)
+			(justify right)
+		)
+	)
 	(hierarchical_label "PB10"
 		(shape input)
@@
 		)
 	)
+	(hierarchical_label "PA6"
+		(shape output)
+		(at 151.13 54.61 180)
+		(fields_autoplaced yes)
+		(effects
+			(font
+				(size 1.27 1.27)
+			)
+			(justify right)
+		)
+	)
 	(hierarchical_label "PA1"
 		(shape output)
@@
 		)
 	)
+	(hierarchical_label "PE0"
+		(shape output)
+		(at 151.13 49.53 180)
+		(fields_autoplaced yes)
+		(effects
+			(font
+				(size 1.27 1.27)
+			)
+			(justify right)
+		)
+	)
 	(hierarchical_label "PE7"
 		(shape input)
@@
 		)
 	)
+	(hierarchical_label "PA7"
+		(shape input)
+		(at 151.13 57.15 180)
+		(fields_autoplaced yes)
+		(effects
+			(font
+				(size 1.27 1.27)
+			)
+			(justify right)
+		)
+	)
+	(hierarchical_label "PE2"
+		(shape input)
+		(at 151.13 62.23 180)
+		(fields_autoplaced yes)
+		(effects
+			(font
+				(size 1.27 1.27)
+			)
+			(justify right)
+		)
+	)
+	(hierarchical_label "PE1"
+		(shape output)
+		(at 151.13 52.07 180)
+		(fields_autoplaced yes)
+		(effects
+			(font
+				(size 1.27 1.27)
+			)
+			(justify right)
+		)
+	)
 	(hierarchical_label "PC4"
 		(shape input)
@@
 			)
 		)
-		(property "Value" "+3.3V"
+		(property "Value" "+3V3"
 			(at 255.27 135.89 0)
 			(effects
@@
 			)
 		)
-		(property "Value" "+3.3V"
+		(property "Value" "+3V3"
 			(at 67.31 26.67 0)
 			(effects
@@
 		(on_board yes)
 		(dnp no)
-		(fields_autoplaced yes)
 		(property "Reference" "U5"
-			(at 173.6441 69.85 0)
+			(at 175.006 69.342 0)
 			(effects
 				(font
@@
 		)
 		(property "Value" "LIS3DH"
-			(at 173.6441 72.39 0)
+			(at 175.006 71.882 0)
 			(effects
 				(font
@@
 			)
 		)
-		(property "Value" "+3.3V"
+		(property "Value" "+3V3"
 			(at 179.07 104.14 0)
 			(effects
@@
 			)
 		)
-		(property "Value" "+3.3V"
+		(property "Value" "+3V3"
 			(at 255.27 24.13 0)
 			(effects

Commit message: Update
Parts:
- added BT2: Li-Ion Battery, symbol Device:Battery
- added C8: 0.47uF, symbol Device:C
- added C9: 1uF, symbol Device:C
- added D3, D4, D5, D6: Load LED (Yellow), symbol Device:LED
- added R10: 10k, symbol Device:R_US
- added R28: 4.7k, symbol Device:R_US
- added R29: 10m, symbol Device:R_US
- added R30, R31, R32, R33: 470, symbol Device:R_US
- added R9: 1.8M, symbol Device:R_US
- added U8: BQ27441-G1, Package_SON:Texas_S-PDSO-N12, symbol Battery_Management:BQ27441-G1
Connections:
- net +3V3: now also R28.1
- net GND: now also BT2.2 (-), C8.2, C9.2, D3.1 (K), D4.1 (K), D5.1 (K), D6.1 (K), R10.2, U8.13 (PAD), U8.3 (V_{SS})
- net PB10: now also U8.2 (SCL)
- net PB11: now also U8.1 (SDA)
- new net: D3.2 (A), R30.2
- new net: D4.2 (A), R31.2
- new net: D5.2 (A), R32.2
- new net: R10.1, R9.2, U8.10 (BIN)
- new net: D6.2 (A), R33.2
- new net +BATT: BT2.1 (+), C9.1, R29.1, U8.6 (BAT), U8.8 (SRP)
- new net GPOUT: R28.2, U8.12 (GPOUT)
- new net VDD: C8.1, R9.1, U8.5 (V_{DD})
- new net VSYS: R29.2, R30.1, R31.1, R32.1, R33.1, U8.7 (SRN)
Other:
- note added: "I2C Address: 0x55"
- note added: "Li-Ion Battery Fuel Gauge"
- note added: "Li-Ion Battery Load"
- note added: "Pull-Up Resistors"
- note added: "Real-Time Clock"
- note removed: "I2C Pullups"
- note removed: "RTC"
- moved on the sheet: BT1, BZ1, C3, C4, C5, C6, C7, D2, Q7, R11, R12, R26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

Commit message: Update
Parts:
- removed D4, D5, D6: Load LED (Yellow), symbol Device:LED
- removed Q7: BC847, Package_TO_SOT_SMD:SOT-23, symbol Transistor_BJT:BC847
- removed R33: 470, symbol Device:R_US
- added Q7, Q8: BC817, Package_TO_SOT_SMD:SOT-23, symbol Transistor_BJT:BC817
- D3: value Load LED (Yellow) -> Battery LED (Yellow)
- R32: value 470 -> 33
Connections:
- net +3V3: now also Q7.3 (C)
- net GND: now also Q8.2 (E)
- net PE7: now also Q7.1 (B)
- net VSYS: no longer R31.1
- net at R31.2: now also Q8.1 (B)
- net at R32.2: now also Q8.3 (C)
- net at BZ1.1 (+): now also Q7.2 (E)
- net VDD renamed +1V8
- new net PE11: R31.1
Other:
- note added: "1Watt"
- note added: "Li-Ion Battery Indicator"
- moved on the sheet: BT1, C3, C4, C5, D2, D3, R11, R12, R30, RV2, SW3, U2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

Commit message: Update
Other:
- note added: "UNUSED"
- moved on the sheet: BT1, BZ1, C3, C4, C5, C6, C7, D2, D3, Q7, Q8, R11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

Commit message: Update
Parts:
- BT2: value Li-Ion Battery -> 4.2V
Connections:
- net +3V0: now reaches BT1.1 (+), U3.14 (VBAT)
Other:
- note added: "CR2032"
- note added: "Li-ion Battery"
- moved on the sheet: C3

Commit message: Update
Parts:
- removed BT1: 3V, symbol Device:Battery_Cell
- removed BT2: 4.2V, symbol Device:Battery
- added J3: LiPo_4.2V, symbol Connector_Generic:Conn_01x02
- added J4: CR2032_3V, symbol Connector_Generic:Conn_01x02
Connections:
- net +3V0: now also J4.1 (Pin_1)
- net +BATT: now also J3.1 (Pin_1)
- net GND: now also J3.2 (Pin_2), J4.2 (Pin_2)
Other:
- note added: "+"
- note added: "-"
- note added: "Socket for Li-ion Battery"
- note removed: "CR2032"
- note removed: "Li-ion Battery"
- moved on the sheet: C3
