File: rjx_training_kit/peripherals.kicad_sch (KiCad schematic)
At the start: 31 parts, among them J3 LiPo_4.2V, J4 CR2032_3V, Q7 BC817, Q8 BC817, SW3 SW_Push, U2 BME280, U3 DS3231M, U5 LIS3DH, U8 BQ27441-G1

Commit message: Update
Parts:
- D2: value User LED (Green) -> LED (Green)
- renumbered J3 to J2, J4 to J3
Connections:
- net +3V3: no longer RV2.3
- new net +3V3A: RV2.3
Other:
- moved on the sheet: C4, C5, D2, R11, R12, SW3, U2

Commit message: Update
Parts:
- removed R28: 4.7k, symbol Device:R_US
- added R13: 4.7k, symbol Device:R_US
- R12: value 470 -> 1.5k
- renumbered C3 to C10, C6 to C11, C7 to C12, C4 to C6, C5 to C7, C9 to C8, C8 to C9, D3 to D2, D2 to D3, J2 to J4, J3 to J5, Q7 to Q1, Q8 to Q2, R11 to R10, R31 to R11, R32 to R14, R27 to R4, R26 to R5, R30 to R6, R9 to R7, R29 to R8, R10 to R9, RV2 to RV1, SW3 to SW2, U2 to U3, U8 to U4, U3 to U5, U5 to U6
Connections:
- net +3V3: now also R13.1
- net GPOUT: no longer names the net of U4.12 (GPOUT)
- net GPOUT: now also R13.2
Other:
- note added: "I2C Pull-Up Resistors"
- note removed: "Pull-Up Resistors"
- note removed: "UNUSED"

Commit message: Update
Parts:
- removed U5: DS3231M, Package_SO:SOIC-16W_7.5x10.3mm_P1.27mm, symbol Timer_RTC:DS3231M
- added C30: C, symbol Device:C
- added D4: BAT54C, Package_TO_SOT_SMD:SOT-23, symbol Diode:BAT54C
- added R15, R8: 300, symbol Device:R_US
- added R16: 2k, symbol Device:R_US
- added R42, R43: 4.7k, symbol Device:R_US
- added U5: PCF8563T, Package_SO:SOIC-8_3.9x4.9mm_P1.27mm, symbol Timer_RTC:PCF8563T
- added Y2: 32.768kHz, symbol Device:Crystal
- C10: value 0.1uF -> 100nF
- R13: renamed from R11; value 470 -> 300
- R14: renamed from R12; value 1.5k -> 2k
- R7: renamed from R6; value 470 -> 300
- renumbered R8 to R10, R9 to R11, R10 to R12, R13 to R17, R14 to R18, R4 to R5, R5 to R6, R7 to R9
Connections:
- net +3V3: now also D4.1; no longer C10.1
- net GND: now also C10.1, C30.2, U5.4 (VSS); no longer C10.2
- net PB10: now also U5.6 (SCL)
- net PB11: now also U5.5 (SDA)
- net PC4: now also R16.1
- net VSYS: no longer R7.1
- net at D2.2 (A): now also R8.2; no longer R7.2
- net at D3.2 (A), R14.2: now also R16.2
- net at Q2.1 (B): now also R15.2; no longer R13.2
- net +3V0: no longer names the net of J5.1 (Pin_1)
- net +3V0: now also D4.2
- new net: R7.2, R8.1
- new net: C10.2, D4.3, R42.1, R43.1, U5.8 (VDD)
- new net: R13.2, R15.1
- new net: C30.1, U5.1 (OSCI), Y2.2
- new net: U5.2 (OSCO), Y2.1
- new net PE12: R42.2, U5.7 (CLKO)
- new net PE13: R43.2, U5.3 (~{INT})
- no-connect marks 3 -> 0
Other:
- note added: "I2C Address: 0x51"
- note removed: "I2C Address: 0x68"
- moved on the sheet: D2, D3, J5, Q2, R12, R13, R14, R18, R7, SW2

Commit message: Update
Parts:
- BZ1: value Buzzer -> 3V_Buzzer
- renumbered C6 to C5, C7 to C6, C8 to C7, C9 to C8, C30 to C9, J4 to J5, J5 to J6, R9 to R10, R10 to R11, R11 to R12, R12 to R13, R13 to R14, R14 to R15, R15 to R16, R16 to R17, R17 to R18, R18 to R19, R42 to R20, R43 to R21, R5 to R6, R6 to R7, R7 to R8, R8 to R9, Y2 to Y1
Connections:
- net PE13 is gone; now on net PE12: R21.2, U5.3 (~{INT})
- net PE12: no longer R20.2, U5.7 (CLKO)
- net VSYS: now also R8.1
- net +3V0: now reaches D4.2, J6.1 (Pin_1)
- new net RTC_CLKO: R20.2, U5.7 (CLKO)
Other:
- note added: "I2C2 Pull-Up Resistors"
- note added: "Note: This circuit speeds up the discharge of the Li-ion battery using a low resistance load."
- note added: "Note: V(BZ1) = V(PE7) - VBE(Q1) = 3.3 - 0.7 = 2.6V"
- note removed: "I2C Pull-Up Resistors"
- moved on the sheet: BZ1, C10, C9, D4, J6, Q1, R20, R21, U5, Y1

Commit message: Update
Parts:
- removed C10, C5, C6: 100nF, symbol Device:C
- removed C9: C, symbol Device:C
- removed D2: Battery LED (Yellow), symbol Device:LED
- removed D4: BAT54C, Package_TO_SOT_SMD:SOT-23, symbol Diode:BAT54C
- removed J6: CR2032_3V, symbol Connector_Generic:Conn_01x02
- removed R11: 10m, symbol Device:R_US
- removed R20: 4.7k, symbol Device:R_US
- removed R8, R9: 300, symbol Device:R_US
- removed U3: BME280, Package_LGA:Bosch_LGA-8_2.5x2.5mm_P0.65mm_ClockwisePinNumbering, symbol Sensor:BME280
- removed U5: PCF8563T, Package_SO:SOIC-8_3.9x4.9mm_P1.27mm, symbol Timer_RTC:PCF8563T
- removed Y1: 32.768kHz, symbol Device:Crystal
- added DS1: WC1602A, Display:WC1602A, symbol Display_Character:WC1602A
- added Q3: BC808, Package_TO_SOT_SMD:SOT-23, symbol Transistor_BJT:BC808
- added Q4: BC817, Package_TO_SOT_SMD:SOT-23, symbol Transistor_BJT:BC817
- added R10: 10m, symbol Device:R_US
- added R12, R13, R14, R15, R16, R18, R19: 270, symbol Device:R_US
- added R23, R27: 1k5, symbol Device:R_US
- added R26: 10k, symbol Device:R_US
- added R28: 300, symbol Device:R_US
- added RV2: 10k, symbol Device:R_Potentiometer_Trim_US
- added U3: TMP1075DGK, Package_SO:VSSOP-8_3x3mm_P0.65mm, symbol Sensor_Temperature:TMP1075DGK
- added U4: MCP2562-E-SN, Package_SO:SOIC-8_3.9x4.9mm_P1.27mm, symbol Interface_CAN_LIN:MCP2562-E-SN
- added U5: BQ24072RGT, Package_DFN_QFN:VQFN-16-1EP_3x3mm_P0.5mm_EP1.6x1.6mm, symbol Battery_Management:BQ24072RGT
- added U7: KCSA02-136, Display_7Segment:KCSC02-136, symbol Display_Character:KCSA02-136
- R17: value 2k -> 270
- R21: value 4.7k -> 10k
- R6, R7: value 4.7k -> 4k7
- R8: renamed from R15; value 2k -> 1k5
- renumbered C7 to C5, C8 to C6, C11 to C7, C12 to C8, D3 to D2, J5 to J4, R12 to R11, R14 to R20, R16 to R22, R18 to R24, R19 to R25, R13 to R5, R10 to R9, U4 to U6, U6 to U8
Connections:
- net PE1 is gone; now on net PA5: U8.9 (INT2)
- net +3V3: now also R21.1, Q3.2 (E)
- net +BATT: no longer U6.8 (SRP)
- net GND: now also DS1.1 (VSS), DS1.5 (R/W), Q4.2 (E), R26.2, RV2.1
- net PA1: now also U8.4 (SPC); no longer RV1.2
- net PA5: no longer U8.4 (SPC)
- net PC4: now also DS1.11 (D4); no longer R17.1, R8.1
- net PC5: now also DS1.12 (D5); no longer R5.2, SW2.2
- net at D2.2 (A), R8.2: no longer R17.2
- net PB10 renamed PB8
- net PB8: now also U3.2 (SCL)
- net PB11 renamed PB9
- net PB9: now also U3.1 (SDA)
- net PE0 renamed PA4
- net PE11 renamed PC13
- net PE12 renamed PA3
- net PA3: now also R23.1
- net PE2 renamed PC8
- net PE7 renamed PB12
- net VSYS: no longer names the net of R25.1
- net VSYS: no longer U6.7 (SRN)
- new net: R18.2, U7.10 (G)
- new net: Q4.1 (B), R27.2
- new net: R13.2, U7.6 (B)
- new net: Q3.1 (B), R23.2
- new net: DS1.15 (LED(+)), R28.1
- new net: DS1.16 (LED(-)), Q4.3 (C)
- new net: Q3.3 (C), U7.3 (CA), U7.8 (CA)
- new net: R15.2, U7.2 (D)
- new net: DS1.3 (VO), RV2.2
- new net: R12.2, U7.7 (A)
- new net: R17.2, U7.9 (F)
- new net: R16.2, U7.1 (E)
- new net: R19.2, U7.5 (DP)
- new net: R14.2, U7.4 (C)
- new net: U5.10 (OUT), U5.11 (OUT)
- new net: U5.17 (VSS), U5.8 (VSS)
- new net: U5.2 (BAT), U5.3 (BAT)
- new net +5V: DS1.2 (VDD), R28.2, RV2.3
- new net PA0: RV1.2
- new net PA11: U4.1 (TXD)
- new net PA12: U4.4 (RXD)
- new net PB0: R12.1
- new net PB1: R13.1
- new net PB13: R8.1
- new net PB14: R5.2, SW2.2
- new net PB15: R26.1, R27.1
- new net PB2: R14.1
- new net PB3: R15.1
- new net PB4: R16.1
- new net PB5: R17.1
- new net PB6: R18.1
- new net PB7: R19.1
- new net PC0: DS1.7 (D0)
- new net PC1: DS1.8 (D1)
- new net PC2: DS1.9 (D2)
- new net PC3: DS1.10 (D3)
- new net PC6: DS1.13 (D6)
- new net PC7: DS1.14 (D7)
- new net PC9: DS1.4 (RS)
- new net PD2: DS1.6 (E)
- new net SRN: U6.7 (SRN)
- new net SRP: U6.8 (SRP)
Other:
- note added: "7 Segment Display"
- note added: "ADC1_IN5"
- note added: "Backlight ON/OFF Control"
- note added: "CAN Transceiver"
- note added: "CAN1_RX"
- note added: "CAN1_TX"
- note added: "I2C1_SCL"
- note added: "I2C1_SDA"
- note added: "LCD"
- note added: "Temperature Sensor"
- note removed: "ADC1_IN1"
- note removed: "I2C Address: 0x51"
- note removed: "I2C Address: 0x76"
- note removed: "I2C2 Pull-Up Resistors"
- note removed: "I2C2_SCL"
- note removed: "I2C2_SDA"
- note removed: "Li-Ion Battery Indicator"
- note removed: "Real-Time Clock"
- note removed: "Temperature & Humidity Sensor"
- moved on the sheet: BZ1, C5, C6, C7, C8, D2, J4, Q1, Q2, R11, R20, R22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

Commit message: Update
Parts:
- added C5: 1uF, symbol Device:C
- added J5: LiPo_4.2V, symbol Connector_Generic:Conn_01x02
- added JP2, JP3, JP?: Jumper_2_Open, symbol Jumper:Jumper_2_Open
- added R9: 1k5, symbol Device:R_US
- BZ1: value 3V_Buzzer -> 5V_Buzzer
- renumbered C5 to C6, C6 to C7, C7 to C8, C8 to C9, Q3 to Q2, Q2 to Q3, R9 to R10, R10 to R11, R11 to R12, R12 to R13, R13 to R14, R14 to R15, R15 to R16, R16 to R17, R17 to R18, R18 to R19, R19 to R20, R23 to R22, R20 to R23, R22 to R24, R24 to R26, R26 to R27, R27 to R28, R28 to R29
Connections:
- net SRP is gone; now on net +BATT: U6.8 (SRP)
- net +3V3: now also JP2.2 (B); no longer Q1.3 (C), Q2.2 (E), R21.1
- net +5V: now also BZ1.1 (+), JP3.2 (B), JP?.2 (B); no longer DS1.2 (VDD), R29.2, RV2.3
- net +BATT: now also R11.2, J5.1 (Pin_1)
- net GND: now also Q1.2 (E), U3.4 (GND), U5.17 (VSS), U5.8 (VSS), C5.2, J5.2 (Pin_2); no longer BZ1.2 (-)
- net PB12: now also R9.1; no longer Q1.1 (B)
- net SRN: now also R11.1, U5.2 (BAT), U5.3 (BAT)
- net at U5.13 (IN): now also C5.1, JP?.1 (A)
- new net: JP2.1 (A), Q2.2 (E), R21.1
- new net: Q1.1 (B), R9.2
- new net: DS1.2 (VDD), JP3.1 (A), R29.2, RV2.3
- new net: BZ1.2 (-), Q1.3 (C)
Other:
- note added: "Charger"
- note added: "Fuel Gauge"
- note added: "I2C Pull-up Resistors"
- note added: "LiPo Battery Sockets"
- note added: "Liquid Crystal Display"
- note added: "Lithium Battery Charging & State-of-charge Measurement"
- note added: "Load"
- note removed: "LCD"
- note removed: "Li-Ion Battery Fuel Gauge"
- note removed: "Li-Ion Battery Load"
- note removed: "Note: V(BZ1) = V(PE7) - VBE(Q1) = 3.3 - 0.7 = 2.6V"
- note removed: "Socket for Li-ion Battery"
- moved on the sheet: BZ1, C6, C7, C8, C9, D2, DS1, J4, Q1, Q2, Q3, Q4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

Commit message: Update
Parts:
- added C12, C13, C14: 100nF, symbol Device:C
- added C7, C8: 4.7uF, symbol Device:C
- added D2: Green, symbol Device:LED
- added D3: Yellow, symbol Device:LED
- added D4: Orange, symbol Device:LED
- added J6: CHG_OUT, symbol Connector:Conn_01x02_Pin
- added J7, J8: CAN_Bus, symbol Connector:Conn_01x02_Pin
- added JP3: Jumper_2_Open, symbol Jumper:Jumper_2_Open
- added R11: 10k, symbol Device:R_US
- added R14, R15, R32, R7, R8: 1.5k, symbol Device:R_US
- added R18: 300, symbol Device:R_US
- added R36: 120, symbol Device:R_US
- added R39: 4.7k, symbol Device:R_US
- added R5: 56k, symbol Device:R_US
- D5: renamed from D2; value LED (Green) -> Green
- R20: renamed from R13; value 270 -> 300
- R21: renamed from R14; value 270 -> 300
- R22: renamed from R15; value 270 -> 300
- R23: renamed from R16; value 270 -> 300
- R24: renamed from R17; value 270 -> 300
- R25: renamed from R18; value 270 -> 300
- R26: renamed from R19; value 270 -> 300
- R27: renamed from R20; value 270 -> 300
- R29: renamed from R22; value 1k5 -> 1.5k
- R31: renamed from R8; value 1k5 -> 1.5k
- R34: renamed from R28; value 1k5 -> 1.5k
- R37: renamed from R7; value 4k7 -> 4.7k
- R38: renamed from R6; value 4k7 -> 4.7k
- R6: renamed from R9; value 1k5 -> 1.5k
- gave numbers to parts that had none: 1
- renumbered C9 to C10, C7 to C11, C8 to C9, JP3 to JP4, Q3 to Q2, Q2 to Q3, R12 to R10, R11 to R12, R23 to R13, R24 to R16, R25 to R17, R26 to R19, R21 to R28, R5 to R30, R27 to R33, R29 to R35, R10 to R9, U5 to U3, U8 to U4, U6 to U5, U7 to U6, U3 to U7, U4 to U8
Connections:
- net +3V3: now also U7.8 (V+), U8.5 (Vio), C12.1, C14.1, R39.1
- net +5V: now also U8.3 (VDD), C13.1
- net +BATT: now also J5.2 (Pin_2); no longer J5.1 (Pin_1)
- net GND: now also J5.1 (Pin_1), U3.15 (TD), U3.4 (~{CE}), U3.6 (EN1), U7.5 (A2), U7.6 (A1), U7.7 (A0), U8.2 (VSS), C12.2, C13.2, C14.2, C7.2, C8.2, J6.2 (Pin_2), R11.2, R5.2, R7.2, R8.2; no longer J5.2 (Pin_2)
- net PA1: now also U7.3 (ALERT), R39.2; no longer U4.4 (SPC)
- net PA11: now also U8.4 (RXD); no longer U8.1 (TXD)
- net PA12: now also U8.1 (TXD); no longer U8.4 (RXD)
- net PB13: now also R32.1
- net SRN: now also C8.1
- net at D5.2 (A), R31.2: now also R32.2
- net at Q2.3 (C), R17.2: now also D4.1 (K)
- net OUT: now reaches R17.1
- net OUT: now also U3.10 (OUT), U3.11 (OUT), U3.5 (EN2), C7.1, J6.1 (Pin_1), R14.1, R15.1, R18.1
- net CANL: now reaches U8.6 (CANL)
- net CANL: now also J7.2 (Pin_2), J8.2 (Pin_2), R36.2
- net CANH: now reaches U8.7 (CANH)
- net CANH: now also J7.1 (Pin_1), J8.1 (Pin_1), JP3.2 (B)
- net PA8: now reaches U8.8 (STBY)
- net at U3.1 (TS): now also R11.1
- net at U3.12 (ILIM): now also R7.1
- net TMR: now reaches U3.14 (TMR)
- net TMR: now also R5.1
- net at U3.16 (ISET): now also R8.1
- net BQ24072_PGOOD: now reaches U3.7 (~{PGOOD})
- net BQ24072_PGOOD: now also D2.1 (K)
- net BQ24072_CHG: now reaches U3.9 (~{CHG})
- net BQ24072_CHG: now also D3.1 (K)
- net PA6 renamed PC11
- net PA7 renamed PC12
- new net: D2.2 (A), R14.2
- new net: JP3.1 (A), R36.1
- new net: D4.2 (A), R18.2
- new net: D3.2 (A), R15.2
- new net PC10: U4.4 (SPC)
Other:
- note added: "1Watt, 1% Tolerance"
- note added: "600mA Charger"
- note added: "CAN_STBY"
- note added: "Connectors"
- note added: "I(CHG) = 600mA I(IN_MAX) = 1A t(MAXCHG) = 7.5 hours"
- note added: "I2C Address: 0x48"
- note added: "I2C/SMBus Pull-up Resistors"
- note added: "I2C1_SMBA"
- note added: "If Jumper is open, the 120-ohm CAN bus termination resistor is disabled."
- note added: "If Jumper is open: 1. All GPIOs in this LCD sub-circuit can be used for other things 2. LCD will be disabled"
- note added: "If Jumper is open: 1. PB0-PB7 can be used for other things 2. 7-segment will be disabled"
- note added: "If Jumper is open: 1. The load at the OUT terminal of the charger will be powered by the battery (BAT) instead. 2. No charging occurs. Battery discharges through an internal FET to power the system load."
- note added: "JST"
- note added: "LED ON: Charging"
- note added: "LED ON: Good power source"
- note added: "Load/Discharge Indicator"
- note added: "More than one CAN bus connector facilitates the connection of multiple devices on the same bus."
- note added: "Note: I(CHG) = Fast charge current I(IN_MAX) = Input current limit t(MAXCHG) = Fast-charge safety timer"
- note added: "SPI3_MISO"
- note added: "SPI3_MOSI"
- note added: "SPI3_SCK"
- note added: "The CHG_OUT and one of the LiPo connectors can be used for testing purposes."
- note added: "This circuit speeds up the discharge of the LiPo battery with a 33-ohm resistor."
- note removed: "Charger"
- note removed: "I2C Pull-up Resistors"
- note removed: "LiPo Battery Sockets"
- note removed: "Load"
- note removed: "Note: This circuit speeds up the discharge of the Li-ion battery using a low resistance load."
- note removed: "SPI1_MISO"
- note removed: "SPI1_MOSI"
- note removed: "SPI1_SCK"
- moved on the sheet: BZ1, C10, C11, C5, C6, C9, D5, DS1, J4, J5, JP1, JP2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

Commit message: Update
Parts:
- renumbered Q1 to Q2, Q2 to Q3, Q3 to Q4, Q4 to Q5, R9 to R10, R10 to R11, R11 to R12, R12 to R13, R13 to R14, R14 to R15, R15 to R16, R16 to R17, R17 to R18, R18 to R19, R19 to R20, R20 to R21, R21 to R22, R22 to R23, R23 to R24, R24 to R25, R25 to R26, R26 to R27, R27 to R28, R28 to R29, R29 to R30, R30 to R31, R31 to R32, R32 to R33, R33 to R34, R34 to R35, R35 to R37, R37 to R38, R38 to R39, R39 to R40, R5 to R6, R6 to R7, R7 to R8, R8 to R9
Other:
- note added: "BATT_DISCHARGE"
- moved on the sheet: BZ1, J4, J5, J6, Q2, R7
