File: rjx_training_kit/power_section.kicad_sch (KiCad schematic)
At the start: 12 parts, among them J1 Barrel_Jack_Switch, J2 USB_B_Mini, SW1 SW_SPDT, U6 MPM3610GQV-P

Commit message: Update
Parts:
- removed C1: 10uF, symbol Device:C_Polarized_US
- removed C2: 22uF, symbol Device:C_Polarized_US
- added C1: 10uF, symbol Device:C
- added C2: 22uF, symbol Device:C
Connections:
- net +3V3: now also C2.1
- net +5V: now also C1.1
- net GND: now also C1.2, C2.2

Commit message: Update
Parts:
- R1: value 330 -> 1.5k
Changed lines of the file:
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@@
 			)
 		)
-		(property "Value" "330"
+		(property "Value" "1.5k"
 			(at 120.65 152.3999 0)
 			(effects

Commit message: Update
Other:
- note added: "Power Supply (Step-Down Converter)"
Changed lines of the file:
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@@
 			(font
 				(size 1.905 1.905)
-				(thickness 0.381)
-				(bold yes)
+				(thickness 0.2381)
 			)
 		)
@@
 		(exclude_from_sim no)
 		(at 232.41 115.57 0)
+		(effects
+			(font
+				(size 1.905 1.905)
+				(thickness 0.2381)
+			)
+		)
+	)
+	(text "5V Sources:  \n1. AC-DC adapter  \n2. USB port"
+		(exclude_from_sim no)
+		(at 31.75 87.122 0)
+		(effects
+			(font
+				(size 1.905 1.905)
+				(thickness 0.2381)
+			)
+			(justify left)
+		)
+	)
+	(text "1"
+		(exclude_from_sim no)
+		(at 246.126 111.76 0)
+		(effects
+			(font
+				(size 1.905 1.905)
+				(thickness 0.2381)
+			)
+		)
+	)
+	(text "R5"
+		(exclude_from_sim no)
+		(at 220.218 107.188 0)
+		(effects
+			(font
+				(size 1.905 1.905)
+				(thickness 0.2381)
+			)
+		)
+	)
+	(text "="
+		(exclude_from_sim no)
+		(at 224.536 106.934 0)
+		(effects
+			(font
+				(size 1.905 1.905)
+			)
+		)
+	)
+	(text "Power Supply (Step-Down Converter)"
+		(exclude_from_sim no)
+		(at 163.068 60.452 0)
 		(effects
 			(font
@@
 				(thickness 0.381)
 				(bold yes)
-			)
-		)
-	)
-	(text "5V Sources:  \n1. AC-DC adapter  \n2. USB port"
-		(exclude_from_sim no)
-		(at 31.75 87.122 0)
-		(effects
-			(font
-				(size 1.905 1.905)
-				(thickness 0.381)
-				(bold yes)
-			)
-			(justify left)
-		)
-	)
-	(text "1"
-		(exclude_from_sim no)
-		(at 246.126 111.76 0)
-		(effects
-			(font
-				(size 1.905 1.905)
-				(thickness 0.381)
-				(bold yes)
-			)
-		)
-	)
-	(text "R5"
-		(exclude_from_sim no)
-		(at 220.218 107.188 0)
-		(effects
-			(font
-				(size 1.905 1.905)
-				(thickness 0.381)
-				(bold yes)
-			)
-		)
-	)
-	(text "="
-		(exclude_from_sim no)
-		(at 224.536 106.934 0)
-		(effects
-			(font
-				(size 1.905 1.905)
 			)
 		)
@@
 			(font
 				(size 1.905 1.905)
-				(thickness 0.381)
-				(bold yes)
+				(thickness 0.2381)
 			)
 		)
@@
 			(font
 				(size 1.905 1.905)
-				(thickness 0.381)
-				(bold yes)
+				(thickness 0.2381)
 			)
 		)
@@
 		(on_board yes)
 		(dnp no)
-		(fields_autoplaced yes)
 		(property "Reference" "R4"
 			(at 198.12 82.5499 0)

Commit message: Update
Other:
- note added: "Power Supply"
- note removed: "Power Supply (Step-Down Converter)"
- moved on the sheet: C1, C2, D1, J1, J2, R1, R2, R3, R4, R5, SW1, U6

Commit message: Update
Changed lines of the file:
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@@
 	)
 	(rectangle
-		(start 52.578 21.59)
+		(start 52.578 32.258)
 		(end 228.854 115.57)
 		(stroke
@@
 	(text "Power Supply"
 		(exclude_from_sim no)
-		(at 136.398 26.67 0)
+		(at 136.398 36.576 0)
 		(effects
 			(font

Commit message: Update
Parts:
- removed C1: 10uF, symbol Device:C
- removed J2: USB_B_Mini, symbol Connector:USB_B_Mini
- removed R4: 75k, symbol Device:R_US
- removed R5: 24k, symbol Device:R_US
- removed U6: MPM3610GQV-P, QFN3p0x5p0x1p6_MPM3610_MNP, symbol mpm3610:MPM3610GQV-P
- added C1, C28: C_Polarized, symbol Device:C_Polarized
- added C29, C30: C, symbol Device:C
- added L1: L, symbol Device:L
- added U6: TLV76133DCY, Package_TO_SOT_SMD:SOT-223-3_TabPin2, symbol Regulator_Linear:TLV76133DCY
- added U7: LM2596S-ADJ, Package_TO_SOT_SMD:TO-263-5_TabPin3, symbol Regulator_Switching:LM2596S-ADJ
- C2: value 22uF -> C
- R2: value 100k -> R_US
- R3: value 39k -> R_US
Connections:
- net +3V3: now also C2.2, R3.2, C28.1, L1.1; no longer C2.1
- net +5V: now also SW1.1 (A), C1.1, C29.1, U6.3 (VI), U7.1 (VIN); no longer R2.2, SW1.2 (B)
- net GND: now also R2.1, C1.2, C28.2, C29.2, C30.2, U6.1 (GND), U7.3 (GND), U7.5 (~{ON}/OFF); no longer C2.2, R3.1
- net at J1.1: now also SW1.2 (B); no longer SW1.1 (A)
- new net: C2.1, R2.2, R3.1, U7.4 (FB)
- new net: L1.2, U7.2 (OUT)
- new net +3V3A: C30.1, U6.2 (VO)
- no-connect marks 8 -> 1
Other:
- note added: "Digital Power Supply"
- note removed: "0.798"
- note removed: "1"
- note removed: "5V Sources: 1. AC-DC adapter 2. USB port"
- note removed: "="
- note removed: "From the MPM3610's datasheet,"
- note removed: "Power Supply"
- note removed: "R4"
- note removed: "R5"
- note removed: "Vout"
- moved on the sheet: D1, J1, R1, SW1
