File: rjx_training_kit/microcontroller.kicad_sch (KiCad schematic)
At the start: 2 parts, among them SW2 SW_Push, U1 STM32F407VGTx

Commit message: Update
Connections:
- net PE2: now reaches U1.1 (PE2)
- net PA5: now reaches U1.30 (PA5)
- net PA6: now reaches U1.31 (PA6)
- net PA7: now reaches U1.32 (PA7)
- net PC4: now reaches U1.33 (PC4)
- net PC5: now reaches U1.34 (PC5)
- net PB0: now reaches U1.35 (PB0)
- net PB1: now reaches U1.36 (PB1)
- net PB2: now reaches U1.37 (PB2)
- net PE7: now reaches U1.38 (PE7)
- net PE8: now reaches U1.39 (PE8)
- net PE9: now reaches U1.40 (PE9)
- net PE10: now reaches U1.41 (PE10)
- net PB10: now reaches U1.47 (PB10)
- net PB11: now reaches U1.48 (PB11)
- net PD11: now reaches U1.58 (PD11)
- net PD12: now reaches U1.59 (PD12)
- net PD13: now reaches U1.60 (PD13)
- net PD14: now reaches U1.61 (PD14)
- net PD15: now reaches U1.62 (PD15)
- net PD0: now reaches U1.81 (PD0)
- net PD1: now reaches U1.82 (PD1)
- net PD2: now reaches U1.83 (PD2)
- net PD3: now reaches U1.84 (PD3)
- net PD4: now reaches U1.85 (PD4)
- net PD5: now reaches U1.86 (PD5)
- net PD6: now reaches U1.87 (PD6)
- net PD7: now reaches U1.88 (PD7)
- net PB3: now reaches U1.89 (PB3)
- net PB4: now reaches U1.90 (PB4)
- net PB5: now reaches U1.91 (PB5)
- net PB6: now reaches U1.92 (PB6)
- net PB7: now reaches U1.93 (PB7)
- net PE0: now reaches U1.97 (PE0)
- net PE1: now reaches U1.98 (PE1)
Other:
- moved on the sheet: SW2, U1

Commit message: Update
Connections:
- net PA1: now reaches U1.24 (PA1)
Changed lines of the file:
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@@
+	(wire
+		(pts
+			(xy 153.67 39.37) (xy 161.29 39.37)
+		)
+		(stroke
+			(width 0)
+			(type default)
+		)
+	)
 	(wire
 		(pts
@@
 		)
 	)
+	(label "PA1"
+		(at 154.94 39.37 0)
+		(fields_autoplaced yes)
+		(effects
+			(font
+				(size 1.27 1.27)
+			)
+			(justify left bottom)
+		)
+	)
 	(label "PB10"
 		(at 160.02 105.41 180)
@@
 		)
 	)
+	(hierarchical_label "PA1"
+		(shape input)
+		(at 161.29 39.37 0)
+		(fields_autoplaced yes)
+		(effects
+			(font
+				(size 1.27 1.27)
+			)
+			(justify left)
+		)
+	)

Commit message: Update
Parts:
- added C10, C11: 2.2uF, symbol Device:C
- added C12: 100nF, symbol Device:C
Connections:
- net GND: now reaches SW2.1
- net GND: now also U1.10 (VSS), U1.20 (VSSA), U1.27 (VSS), U1.74 (VSS), U1.99 (VSS), C10.2, C11.2, C12.2
- net NRST: now reaches SW2.2
- net NRST: now also U1.14 (NRST), C12.1
- net PE11: now reaches U1.42 (PE11)
- net at U1.49 (VCAP_1): now also C10.1
- net at U1.73 (VCAP_2): now also C11.1
Other:
- note added: "BOOT Pins"
- note added: "BOOT1"
- note added: "External Reset Circuit"
- moved on the sheet: SW2, U1

Commit message: Update
Parts:
- added R38, R39: 10k, symbol Device:R_US
Connections:
- net GND: now also R38.2
- net PB2: now also R39.2
- net BOOT0: now reaches U1.94 (BOOT0)
- net BOOT0: now also R38.1
- new net +3V3: R39.1
Other:
- note added: ". Default BOOT[1:0] = "10" . MCU boots from flash memory"
- moved on the sheet: C12, SW2

Commit message: Update
Parts:
- added C13: 4.7uF, symbol Device:C
- added C14, C15, C16, C19, C20, C21, C22, C23: 100nF, symbol Device:C
- added C17, C18: 1uF, symbol Device:C
- added C24, C25, C26, C27: C, symbol Device:C
- added FB1: FerriteBead_Small, symbol Device:FerriteBead_Small
- added Y1: 8MHz, symbol Device:Crystal
- added Y2: 32.768kHz, symbol Device:Crystal
Connections:
- net +3V3: now also U1.100 (VDD), U1.11 (VDD), U1.19 (VDD), U1.28 (VDD), U1.50 (VDD), U1.75 (VDD), C13.1, C14.1, C15.1, C16.1, C19.1, C22.1, C23.1, FB1.1
- net GND: now also C13.2, C14.2, C15.2, C16.2, C17.2, C18.2, C19.2, C20.2, C21.2, C22.2, C23.2, C24.1, C25.1, C26.1, C27.1
- net PH0: now reaches U1.12 (PH0)
- net PH0: now also C24.2, Y1.1
- net PH1: now reaches U1.13 (PH1)
- net PH1: now also C25.2, Y1.2
- net VDDA: now reaches U1.21 (VREF+)
- net VDDA: now also U1.22 (VDDA), C17.1, C18.1, C20.1, C21.1, FB1.2
- net +3V0: now reaches U1.6 (VBAT)
- net PC14: now reaches U1.8 (PC14)
- net PC14: now also C26.2, Y2.1
- net PC15: now reaches U1.9 (PC15)
- net PC15: now also C27.2, Y2.2
Other:
- note added: "100nF decoupling capacitor per VDD"
- note added: "External Oscillators"
- note added: "HSE"
- note added: "LSE"
- note added: "OSC32_IN"
- note added: "OSC32_OUT"
- note added: "OSC_IN"
- note added: "OSC_OUT"
- note added: "Power Supply Scheme"
- moved on the sheet: C10, C11, C12, R38, R39, SW2, U1

Commit message: Update
Connections:
- net PC0: now reaches U1.15 (PC0)
- net PC1: now reaches U1.16 (PC1)
- net PC2: now reaches U1.17 (PC2)
- net PC3: now reaches U1.18 (PC3)
- net PE3: now reaches U1.2 (PE3)
- net PA0: now reaches U1.23 (PA0)
- net PA2: now reaches U1.25 (PA2)
- net PA3: now reaches U1.26 (PA3)
- net PA4: now reaches U1.29 (PA4)
- net PE4: now reaches U1.3 (PE4)
- net PE5: now reaches U1.4 (PE5)
- net PE12: now reaches U1.43 (PE12)
- net PE13: now reaches U1.44 (PE13)
- net PE14: now reaches U1.45 (PE14)
- net PE15: now reaches U1.46 (PE15)
- net PE6: now reaches U1.5 (PE6)
- net PB12: now reaches U1.51 (PB12)
- net PB13: now reaches U1.52 (PB13)
- net PB14: now reaches U1.53 (PB14)
- net PB15: now reaches U1.54 (PB15)
- net PD8: now reaches U1.55 (PD8)
- net PD9: now reaches U1.56 (PD9)
- net PD10: now reaches U1.57 (PD10)
- net PC6: now reaches U1.63 (PC6)
- net PC7: now reaches U1.64 (PC7)
- net PC8: now reaches U1.65 (PC8)
- net PC9: now reaches U1.66 (PC9)
- net PA8: now reaches U1.67 (PA8)
- net PA9: now reaches U1.68 (PA9)
- net PA10: now reaches U1.69 (PA10)
- net PC13: now reaches U1.7 (PC13)
- net PA11: now reaches U1.70 (PA11)
- net PA12: now reaches U1.71 (PA12)
- net PA13: now reaches U1.72 (PA13)
- net PA14: now reaches U1.76 (PA14)
- net PA15: now reaches U1.77 (PA15)
- net PC10: now reaches U1.78 (PC10)
- net PC11: now reaches U1.79 (PC11)
- net PC12: now reaches U1.80 (PC12)
- net PB8: now reaches U1.95 (PB8)
- net PB9: now reaches U1.96 (PB9)

Commit message: Update
Parts:
- removed FB1: FerriteBead_Small, symbol Device:FerriteBead_Small
- added C31: 100nF, symbol Device:C
- C17: value 1uF -> 100nF
- C23: value 100nF -> 1uF
Connections:
- net +3V0: now also C31.1
- net +3V3: now also C17.1, C21.1; no longer C22.1, C23.1
- net GND: now also C31.2
- net VDDA renamed +3V3A
- net +3V3A: now also C22.1, C23.1; no longer C17.1, C21.1
Other:
- note added: "High-Speed External Oscillator"
- note added: "Low-Speed External Oscillator"
- note removed: "100nF decoupling capacitor per VDD"
- note removed: "External Oscillators"
- note removed: "HSE"
- note removed: "LSE"
- note removed: "Power Supply Scheme"
- moved on the sheet: C10, C11, C12, C24, C25, C26, C27, R38, R39, SW2, U1, Y1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

Commit message: Update
Parts:
- removed C12, C31: 100nF, symbol Device:C
- removed C24, C25, C26: C, symbol Device:C
- removed R38: 10k, symbol Device:R_US
- removed SW2: SW_Push, symbol Switch:SW_Push
- removed Y2: 32.768kHz, symbol Device:Crystal
- added C16: 100nF, symbol Device:C
- added C18, C20: C, symbol Device:C
- added R15: 10k, symbol Device:R_US
- added SW3: SW_Push, symbol Switch:SW_Push
- C27: value C -> 100nF
- renumbered C18 to C13, C13 to C14, C20 to C15, C14 to C17, C15 to C19, C16 to C21, C10 to C22, C17 to C23, C11 to C24, C19 to C25, C21 to C26, C22 to C28, C23 to C29, R39 to R16, U1 to U7
Connections:
- net +3V0 is gone; now on net +3V3: U7.6 (VBAT)
- net +3V3: now also C27.1
- net BOOT0: now also R15.1
- net GND: now also C27.2, C16.2, C18.1, C20.1, R15.2, SW3.1; no longer C27.1
- net NRST: now also C16.1, SW3.2
- net PC15: no longer C27.2
- net PH0: no longer names the net of U7.12 (PH0), Y1.1
- net PH0: now also C18.2
- net PH1: no longer names the net of U7.13 (PH1), Y1.2
- net PH1: now also C20.2
Other:
- note removed: "BOOT Pins"
- note removed: "External Reset Circuit"
- note removed: "High-Speed External Oscillator"
- note removed: "Low-Speed External Oscillator"
- note removed: "OSC32_IN"
- note removed: "OSC32_OUT"
- note removed: "OSC_IN"
- note removed: "OSC_OUT"
- moved on the sheet: C13, C14, C15, C17, C19, C21, C22, C23, C24, C25, C26, C28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
