File: rjx_training_kit/microcontroller.kicad_sch (KiCad schematic)
At the start: 22 parts, among them SW3 SW_Push, U7 STM32F407VGTx, Y1 8MHz

Commit message: Update
Parts:
- renumbered R15 to R19, R16 to R20
Changed lines of the file:
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@@
 		(on_board yes)
 		(dnp no)
-		(property "Reference" "#PWR066"
+		(property "Reference" "#PWR065"
 			(at 157.48 39.37 0)
 			(effects
@@
 			(project "rjx_training_kit"
 				(path "/c10d0f5f-1570-4ced-80f8-bf69ea514c66/6ff37231-b90f-440e-bce5-b002d3bf6e3d"
-					(reference "#PWR066")
+					(reference "#PWR065")
 					(unit 1)
 				)
@@
 		(on_board yes)
 		(dnp no)
-		(property "Reference" "#PWR062"
+		(property "Reference" "#PWR061"
 			(at 116.84 39.37 0)
 			(effects
@@
 			(project "rjx_training_kit"
 				(path "/c10d0f5f-1570-4ced-80f8-bf69ea514c66/6ff37231-b90f-440e-bce5-b002d3bf6e3d"
-					(reference "#PWR062")
+					(reference "#PWR061")
 					(unit 1)
 				)
@@
 		(on_board yes)
 		(dnp no)
-		(property "Reference" "#PWR052"
+		(property "Reference" "#PWR051"
 			(at 59.69 63.5 0)
 			(effects
@@
 			(project "rjx_training_kit"
 				(path "/c10d0f5f-1570-4ced-80f8-bf69ea514c66/6ff37231-b90f-440e-bce5-b002d3bf6e3d"
-					(reference "#PWR052")
+					(reference "#PWR051")
 					(unit 1)
 				)
@@
 		(on_board yes)
 		(dnp no)
-		(property "Reference" "#PWR048"
+		(property "Reference" "#PWR047"
 			(at 48.26 64.77 0)
 			(effects
@@
 			(project "rjx_training_kit"
 				(path "/c10d0f5f-1570-4ced-80f8-bf69ea514c66/6ff37231-b90f-440e-bce5-b002d3bf6e3d"
-					(reference "#PWR048")
+					(reference "#PWR047")
 					(unit 1)
 				)
@@
 		(on_board yes)
 		(dnp no)
-		(property "Reference" "#PWR063"
+		(property "Reference" "#PWR062"
 			(at 128.27 39.37 0)
 			(effects
@@
 			(project "rjx_training_kit"
 				(path "/c10d0f5f-1570-4ced-80f8-bf69ea514c66/6ff37231-b90f-440e-bce5-b002d3bf6e3d"
-					(reference "#PWR063")
+					(reference "#PWR062")
 					(unit 1)
 				)
@@
 		(on_board yes)
 		(dnp no)
-		(property "Reference" "R15"
+		(property "Reference" "R19"
 			(at 94.488 50.8 0)
 			(effects
@@
 			(project ""
 				(path "/c10d0f5f-1570-4ced-80f8-bf69ea514c66/6ff37231-b90f-440e-bce5-b002d3bf6e3d"
-					(reference "R15")
+					(reference "R19")
 					(unit 1)
 				)
@@
 		(on_board yes)
 		(dnp no)
-		(property "Reference" "#PWR058"
+		(property "Reference" "#PWR057"
 			(at 93.98 39.37 0)
 			(effects
@@
 			(project "rjx_training_kit"
 				(path "/c10d0f5f-1570-4ced-80f8-bf69ea514c66/6ff37231-b90f-440e-bce5-b002d3bf6e3d"
-					(reference "#PWR058")
+					(reference "#PWR057")
 					(unit 1)
 				)
@@
 		(on_board yes)
 		(dnp no)
-		(property "Reference" "#PWR059"
+		(property "Reference" "#PWR058"
 			(at 99.06 180.34 0)
 			(effects
@@
 			(project "rjx_training_kit"
 				(path "/c10d0f5f-1570-4ced-80f8-bf69ea514c66/6ff37231-b90f-440e-bce5-b002d3bf6e3d"
-					(reference "#PWR059")
+					(reference "#PWR058")
 					(unit 1)
 				)
@@
 		(on_board yes)
 		(dnp no)
-		(property "Reference" "#PWR064"
+		(property "Reference" "#PWR063"
 			(at 138.43 196.85 0)
 			(effects
@@
 			(project "rjx_training_kit"
 				(path "/c10d0f5f-1570-4ced-80f8-bf69ea514c66/6ff37231-b90f-440e-bce5-b002d3bf6e3d"
-					(reference "#PWR064")
+					(reference "#PWR063")
 					(unit 1)
 				)
@@
 		(on_board yes)
 		(dnp no)
-		(property "Reference" "#PWR068"
+		(property "Reference" "#PWR067"
 			(at 167.64 39.37 0)
 			(effects
@@
 			(project "rjx_training_kit"
 				(path "/c10d0f5f-1570-4ced-80f8-bf69ea514c66/6ff37231-b90f-440e-bce5-b002d3bf6e3d"
-					(reference "#PWR068")
+					(reference "#PWR067")
 					(unit 1)
 				)
@@
 		(on_board yes)
 		(dnp no)
-		(property "Reference" "#PWR054"
+		(property "Reference" "#PWR053"
 			(at 71.12 39.37 0)
 			(effects
@@
 			(project "rjx_training_kit"
 				(path "/c10d0f5f-1570-4ced-80f8-bf69ea514c66/6ff37231-b90f-440e-bce5-b002d3bf6e3d"
-					(reference "#PWR054")
+					(reference "#PWR053")
 					(unit 1)
 				)
@@
 		(on_board yes)
 		(dnp no)
-		(property "Reference" "#PWR055"
+		(property "Reference" "#PWR054"
 			(at 81.28 101.6 0)
 			(effects
@@
 			(project "rjx_training_kit"
 				(path "/c10d0f5f-1570-4ced-80f8-bf69ea514c66/6ff37231-b90f-440e-bce5-b002d3bf6e3d"
-					(reference "#PWR055")
+					(reference "#PWR054")
 					(unit 1)
 				)
@@
 		(on_board yes)
 		(dnp no)
-		(property "Reference" "#PWR056"
+		(property "Reference" "#PWR055"
 			(at 82.55 39.37 0)
 			(effects
@@
 			(project "rjx_training_kit"
 				(path "/c10d0f5f-1570-4ced-80f8-bf69ea514c66/6ff37231-b90f-440e-bce5-b002d3bf6e3d"
-					(reference "#PWR056")
+					(reference "#PWR055")
 					(unit 1)
 				)
@@
 		(on_board yes)
 		(dnp no)
-		(property "Reference" "#PWR049"
+		(property "Reference" "#PWR048"
 			(at 48.26 82.55 0)
 			(effects
@@
 			(project "rjx_training_kit"
 				(path "/c10d0f5f-1570-4ced-80f8-bf69ea514c66/6ff37231-b90f-440e-bce5-b002d3bf6e3d"
-					(reference "#PWR049")
+					(reference "#PWR048")
 					(unit 1)
 				)
@@
 		(on_board yes)
 		(dnp no)
-		(property "Reference" "#PWR051"
+		(property "Reference" "#PWR050"
 			(at 59.69 39.37 0)
 			(effects
@@
 			(project "rjx_training_kit"
 				(path "/c10d0f5f-1570-4ced-80f8-bf69ea514c66/6ff37231-b90f-440e-bce5-b002d3bf6e3d"
-					(reference "#PWR051")
+					(reference "#PWR050")
 					(unit 1)
 				)
@@
 		(on_board yes)
 		(dnp no)
-		(property "Reference" "#PWR057"
+		(property "Reference" "#PWR056"
 			(at 92.71 63.5 0)
 			(effects
@@
 			(project "rjx_training_kit"
 				(path "/c10d0f5f-1570-4ced-80f8-bf69ea514c66/6ff37231-b90f-440e-bce5-b002d3bf6e3d"
-					(reference "#PWR057")
+					(reference "#PWR056")
 					(unit 1)
 				)
@@
 		(on_board yes)
 		(dnp no)
-		(property "Reference" "#PWR067"
+		(property "Reference" "#PWR066"
 			(at 167.64 25.4 0)
 			(effects
@@
 			(project "rjx_training_kit"
 				(path "/c10d0f5f-1570-4ced-80f8-bf69ea514c66/6ff37231-b90f-440e-bce5-b002d3bf6e3d"
-					(reference "#PWR067")
+					(reference "#PWR066")
 					(unit 1)
 				)
@@
 		(on_board yes)
 		(dnp no)
-		(property "Reference" "#PWR060"
+		(property "Reference" "#PWR059"
 			(at 105.41 39.37 0)
 			(effects
@@
 			(project "rjx_training_kit"
 				(path "/c10d0f5f-1570-4ced-80f8-bf69ea514c66/6ff37231-b90f-440e-bce5-b002d3bf6e3d"
-					(reference "#PWR060")
+					(reference "#PWR059")
 					(unit 1)
 				)
@@
 		(on_board yes)
 		(dnp no)
-		(property "Reference" "R16"
+		(property "Reference" "R20"
 			(at 181.864 91.44 0)
 			(effects
@@
 			(project ""
 				(path "/c10d0f5f-1570-4ced-80f8-bf69ea514c66/6ff37231-b90f-440e-bce5-b002d3bf6e3d"
-					(reference "R16")
+					(reference "R20")
 					(unit 1)
 				)
@@
 		(on_board yes)
 		(dnp no)
-		(property "Reference" "#PWR061"
+		(property "Reference" "#PWR060"
 			(at 110.49 180.34 0)
 			(effects
@@
 			(project ""
 				(path "/c10d0f5f-1570-4ced-80f8-bf69ea514c66/6ff37231-b90f-440e-bce5-b002d3bf6e3d"
-					(reference "#PWR061")
+					(reference "#PWR060")
 					(unit 1)
 				)
@@
 		(on_board yes)
 		(dnp no)
-		(property "Reference" "#PWR053"
+		(property "Reference" "#PWR052"
 			(at 59.69 82.55 0)
 			(effects
@@
 			(project "rjx_training_kit"
 				(path "/c10d0f5f-1570-4ced-80f8-bf69ea514c66/6ff37231-b90f-440e-bce5-b002d3bf6e3d"
-					(reference "#PWR053")
+					(reference "#PWR052")
 					(unit 1)
 				)
@@
 		(on_board yes)
 		(dnp no)
-		(property "Reference" "#PWR065"
+		(property "Reference" "#PWR064"
 			(at 139.7 39.37 0)
 			(effects
@@
 			(project "rjx_training_kit"
 				(path "/c10d0f5f-1570-4ced-80f8-bf69ea514c66/6ff37231-b90f-440e-bce5-b002d3bf6e3d"
-					(reference "#PWR065")
+					(reference "#PWR064")
 					(unit 1)
 				)
@@
 		(on_board yes)
 		(dnp no)
-		(property "Reference" "#PWR050"
+		(property "Reference" "#PWR049"
 			(at 59.69 25.4 0)
 			(effects
@@
 			(project "rjx_training_kit"
 				(path "/c10d0f5f-1570-4ced-80f8-bf69ea514c66/6ff37231-b90f-440e-bce5-b002d3bf6e3d"
-					(reference "#PWR050")
+					(reference "#PWR049")
 					(unit 1)
 				)
@@
 		(on_board yes)
 		(dnp no)
-		(property "Reference" "#PWR069"
+		(property "Reference" "#PWR068"
 			(at 180.34 90.17 0)
 			(effects
@@
 			(project "rjx_training_kit"
 				(path "/c10d0f5f-1570-4ced-80f8-bf69ea514c66/6ff37231-b90f-440e-bce5-b002d3bf6e3d"
-					(reference "#PWR069")
+					(reference "#PWR068")
 					(unit 1)
 				)

Commit message: Update
Parts:
- renumbered R19 to R22, R20 to R23, Y1 to Y2
Other:
- note added: "By default, BOOT1 = 1 and BOOT 0 = 0. This configuration makes the MCU boot from flash memory."
- note removed: ". Default BOOT[1:0] = "10" . MCU boots from flash memory"
Changed lines of the file:
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@@
 		)
 	)
-	(text ". Default BOOT[1:0] = \"10\"\n. MCU boots from flash memory"
+	(text "By default, BOOT1 = 1 and BOOT 0 = 0.\nThis configuration makes the MCU boot from flash memory."
 		(exclude_from_sim no)
-		(at 225.044 126.238 0)
+		(at 188.722 108.204 0)
 		(effects
 			(font
-				(size 1.905 1.905)
+				(size 1.27 1.27)
 				(thickness 0.2381)
 			)
@@
 		(on_board yes)
 		(dnp no)
-		(property "Reference" "#PWR065"
+		(property "Reference" "#PWR075"
 			(at 157.48 39.37 0)
 			(effects
@@
 			(project "rjx_training_kit"
 				(path "/c10d0f5f-1570-4ced-80f8-bf69ea514c66/6ff37231-b90f-440e-bce5-b002d3bf6e3d"
-					(reference "#PWR065")
+					(reference "#PWR075")
 					(unit 1)
 				)
@@
 		(on_board yes)
 		(dnp no)
-		(property "Reference" "Y1"
+		(property "Reference" "Y2"
 			(at 80.01 73.406 0)
 			(effects
@@
 			(project "rjx_training_kit"
 				(path "/c10d0f5f-1570-4ced-80f8-bf69ea514c66/6ff37231-b90f-440e-bce5-b002d3bf6e3d"
-					(reference "Y1")
+					(reference "Y2")
 					(unit 1)
 				)
@@
 		(on_board yes)
 		(dnp no)
-		(property "Reference" "#PWR061"
+		(property "Reference" "#PWR071"
 			(at 116.84 39.37 0)
 			(effects
@@
 			(project "rjx_training_kit"
 				(path "/c10d0f5f-1570-4ced-80f8-bf69ea514c66/6ff37231-b90f-440e-bce5-b002d3bf6e3d"
-					(reference "#PWR061")
+					(reference "#PWR071")
 					(unit 1)
 				)
@@
 		(on_board yes)
 		(dnp no)
-		(property "Reference" "#PWR051"
+		(property "Reference" "#PWR061"
 			(at 59.69 63.5 0)
 			(effects
@@
 			(project "rjx_training_kit"
 				(path "/c10d0f5f-1570-4ced-80f8-bf69ea514c66/6ff37231-b90f-440e-bce5-b002d3bf6e3d"
-					(reference "#PWR051")
+					(reference "#PWR061")
 					(unit 1)
 				)
@@
 		(on_board yes)
 		(dnp no)
-		(property "Reference" "#PWR047"
+		(property "Reference" "#PWR057"
 			(at 48.26 64.77 0)
 			(effects
@@
 			(project "rjx_training_kit"
 				(path "/c10d0f5f-1570-4ced-80f8-bf69ea514c66/6ff37231-b90f-440e-bce5-b002d3bf6e3d"
-					(reference "#PWR047")
+					(reference "#PWR057")
 					(unit 1)
 				)
@@
 		(on_board yes)
 		(dnp no)
-		(property "Reference" "#PWR062"
+		(property "Reference" "#PWR072"
 			(at 128.27 39.37 0)
 			(effects
@@
 			(project "rjx_training_kit"
 				(path "/c10d0f5f-1570-4ced-80f8-bf69ea514c66/6ff37231-b90f-440e-bce5-b002d3bf6e3d"
-					(reference "#PWR062")
+					(reference "#PWR072")
 					(unit 1)
 				)
@@
 		(on_board yes)
 		(dnp no)
-		(property "Reference" "R19"
+		(property "Reference" "R22"
 			(at 94.488 50.8 0)
 			(effects
@@
 			(project ""
 				(path "/c10d0f5f-1570-4ced-80f8-bf69ea514c66/6ff37231-b90f-440e-bce5-b002d3bf6e3d"
-					(reference "R19")
+					(reference "R22")
 					(unit 1)
 				)
@@
 		(on_board yes)
 		(dnp no)
-		(property "Reference" "#PWR057"
+		(property "Reference" "#PWR067"
 			(at 93.98 39.37 0)
 			(effects
@@
 			(project "rjx_training_kit"
 				(path "/c10d0f5f-1570-4ced-80f8-bf69ea514c66/6ff37231-b90f-440e-bce5-b002d3bf6e3d"
-					(reference "#PWR057")
+					(reference "#PWR067")
 					(unit 1)
 				)
@@
 		(on_board yes)
 		(dnp no)
-		(property "Reference" "#PWR058"
+		(property "Reference" "#PWR068"
 			(at 99.06 180.34 0)
 			(effects
@@
 			(project "rjx_training_kit"
 				(path "/c10d0f5f-1570-4ced-80f8-bf69ea514c66/6ff37231-b90f-440e-bce5-b002d3bf6e3d"
-					(reference "#PWR058")
+					(reference "#PWR068")
 					(unit 1)
 				)
@@
 		(on_board yes)
 		(dnp no)
-		(property "Reference" "#PWR063"
+		(property "Reference" "#PWR073"
 			(at 138.43 196.85 0)
 			(effects
@@
 			(project "rjx_training_kit"
 				(path "/c10d0f5f-1570-4ced-80f8-bf69ea514c66/6ff37231-b90f-440e-bce5-b002d3bf6e3d"
-					(reference "#PWR063")
+					(reference "#PWR073")
 					(unit 1)
 				)
@@
 		(on_board yes)
 		(dnp no)
-		(property "Reference" "#PWR067"
+		(property "Reference" "#PWR077"
 			(at 167.64 39.37 0)
 			(effects
@@
 			(project "rjx_training_kit"
 				(path "/c10d0f5f-1570-4ced-80f8-bf69ea514c66/6ff37231-b90f-440e-bce5-b002d3bf6e3d"
-					(reference "#PWR067")
+					(reference "#PWR077")
 					(unit 1)
 				)
@@
 		(on_board yes)
 		(dnp no)
-		(property "Reference" "#PWR053"
+		(property "Reference" "#PWR063"
 			(at 71.12 39.37 0)
 			(effects
@@
 			(project "rjx_training_kit"
 				(path "/c10d0f5f-1570-4ced-80f8-bf69ea514c66/6ff37231-b90f-440e-bce5-b002d3bf6e3d"
-					(reference "#PWR053")
+					(reference "#PWR063")
 					(unit 1)
 				)
@@
 		(on_board yes)
 		(dnp no)
-		(property "Reference" "#PWR054"
+		(property "Reference" "#PWR064"
 			(at 81.28 101.6 0)
 			(effects
@@
 			(project "rjx_training_kit"
 				(path "/c10d0f5f-1570-4ced-80f8-bf69ea514c66/6ff37231-b90f-440e-bce5-b002d3bf6e3d"
-					(reference "#PWR054")
+					(reference "#PWR064")
 					(unit 1)
 				)
@@
 		(on_board yes)
 		(dnp no)
-		(property "Reference" "#PWR055"
+		(property "Reference" "#PWR065"
 			(at 82.55 39.37 0)
 			(effects
@@
 			(project "rjx_training_kit"
 				(path "/c10d0f5f-1570-4ced-80f8-bf69ea514c66/6ff37231-b90f-440e-bce5-b002d3bf6e3d"
-					(reference "#PWR055")
+					(reference "#PWR065")
 					(unit 1)
 				)
@@
 		(on_board yes)
 		(dnp no)
-		(property "Reference" "#PWR048"
+		(property "Reference" "#PWR058"
 			(at 48.26 82.55 0)
 			(effects
@@
 			(project "rjx_training_kit"
 				(path "/c10d0f5f-1570-4ced-80f8-bf69ea514c66/6ff37231-b90f-440e-bce5-b002d3bf6e3d"
-					(reference "#PWR048")
+					(reference "#PWR058")
 					(unit 1)
 				)
@@
 		(on_board yes)
 		(dnp no)
-		(property "Reference" "#PWR050"
+		(property "Reference" "#PWR060"
 			(at 59.69 39.37 0)
 			(effects
@@
 			(project "rjx_training_kit"
 				(path "/c10d0f5f-1570-4ced-80f8-bf69ea514c66/6ff37231-b90f-440e-bce5-b002d3bf6e3d"
-					(reference "#PWR050")
+					(reference "#PWR060")
 					(unit 1)
 				)
@@
 		(on_board yes)
 		(dnp no)
-		(property "Reference" "#PWR056"
+		(property "Reference" "#PWR066"
 			(at 92.71 63.5 0)
 			(effects
@@
 			(project "rjx_training_kit"
 				(path "/c10d0f5f-1570-4ced-80f8-bf69ea514c66/6ff37231-b90f-440e-bce5-b002d3bf6e3d"
-					(reference "#PWR056")
+					(reference "#PWR066")
 					(unit 1)
 				)
@@
 		(on_board yes)
 		(dnp no)
-		(property "Reference" "#PWR066"
+		(property "Reference" "#PWR076"
 			(at 167.64 25.4 0)
 			(effects
@@
 			(project "rjx_training_kit"
 				(path "/c10d0f5f-1570-4ced-80f8-bf69ea514c66/6ff37231-b90f-440e-bce5-b002d3bf6e3d"
-					(reference "#PWR066")
+					(reference "#PWR076")
 					(unit 1)
 				)
@@
 		(on_board yes)
 		(dnp no)
-		(property "Reference" "#PWR059"
+		(property "Reference" "#PWR069"
 			(at 105.41 39.37 0)
 			(effects
@@
 			(project "rjx_training_kit"
 				(path "/c10d0f5f-1570-4ced-80f8-bf69ea514c66/6ff37231-b90f-440e-bce5-b002d3bf6e3d"
-					(reference "#PWR059")
+					(reference "#PWR069")
 					(unit 1)
 				)
@@
 		(on_board yes)
 		(dnp no)
-		(property "Reference" "R20"
+		(property "Reference" "R23"
 			(at 181.864 91.44 0)
 			(effects
@@
 			(project ""
 				(path "/c10d0f5f-1570-4ced-80f8-bf69ea514c66/6ff37231-b90f-440e-bce5-b002d3bf6e3d"
-					(reference "R20")
+					(reference "R23")
 					(unit 1)
 				)
@@
 		(on_board yes)
 		(dnp no)
-		(property "Reference" "#PWR060"
+		(property "Reference" "#PWR070"
 			(at 110.49 180.34 0)
 			(effects
@@
 			(project ""
 				(path "/c10d0f5f-1570-4ced-80f8-bf69ea514c66/6ff37231-b90f-440e-bce5-b002d3bf6e3d"
-					(reference "#PWR060")
+					(reference "#PWR070")
 					(unit 1)
 				)
@@
 		(on_board yes)
 		(dnp no)
-		(property "Reference" "#PWR052"
+		(property "Reference" "#PWR062"
 			(at 59.69 82.55 0)
 			(effects
@@
 			(project "rjx_training_kit"
 				(path "/c10d0f5f-1570-4ced-80f8-bf69ea514c66/6ff37231-b90f-440e-bce5-b002d3bf6e3d"
-					(reference "#PWR052")
+					(reference "#PWR062")
 					(unit 1)
 				)
@@
 		(on_board yes)
 		(dnp no)
-		(property "Reference" "#PWR064"
+		(property "Reference" "#PWR074"
 			(at 139.7 39.37 0)
 			(effects
@@
 			(project "rjx_training_kit"
 				(path "/c10d0f5f-1570-4ced-80f8-bf69ea514c66/6ff37231-b90f-440e-bce5-b002d3bf6e3d"
-					(reference "#PWR064")
+					(reference "#PWR074")
 					(unit 1)
 				)
@@
 		(on_board yes)
 		(dnp no)
-		(property "Reference" "#PWR049"
+		(property "Reference" "#PWR059"
 			(at 59.69 25.4 0)
 			(effects
@@
 			(project "rjx_training_kit"
 				(path "/c10d0f5f-1570-4ced-80f8-bf69ea514c66/6ff37231-b90f-440e-bce5-b002d3bf6e3d"
-					(reference "#PWR049")
+					(reference "#PWR059")
 					(unit 1)
 				)
@@
 		(on_board yes)
 		(dnp no)
-		(property "Reference" "#PWR068"
+		(property "Reference" "#PWR078"
 			(at 180.34 90.17 0)
 			(effects
@@
 			(project "rjx_training_kit"
 				(path "/c10d0f5f-1570-4ced-80f8-bf69ea514c66/6ff37231-b90f-440e-bce5-b002d3bf6e3d"
-					(reference "#PWR068")
+					(reference "#PWR078")
 					(unit 1)
 				)

Commit message: Update
Parts:
- removed C22, C24: 2.2uF, symbol Device:C
- removed R23: 10k, symbol Device:R_US
- removed U7: STM32F407VGTx, Package_QFP:LQFP-100_14x14mm_P0.5mm, symbol MCU_ST_STM32F4:STM32F407VGTx
- added U9: STM32L431RCTx, Package_QFP:LQFP-64_10x10mm_P0.5mm, symbol MCU_ST_STM32L4:STM32L431RCTx
- renumbered C14 to C10, C15 to C11, C16 to C12, C17 to C13, C18 to C14, C19 to C15, C20 to C16, C21 to C17, C23 to C18, C25 to C19, C26 to C20, C27 to C21, C28 to C22, C29 to C23, C13 to C9, R22 to R29, Y2 to Y1
Connections:
- new net: U9.18 (VSS), U9.31 (VSS), U9.47 (VSS), U9.63 (VSS)
Other:
- note removed: "BOOT1"
- note removed: "By default, BOOT1 = 1 and BOOT 0 = 0. This configuration makes the MCU boot from flash memory."

Commit message: Update
Parts:
- renumbered C9 to C10, C10 to C11, C11 to C12, C12 to C13, C13 to C14, C14 to C15, C15 to C16, C16 to C17, C17 to C18, C18 to C19, C19 to C20, C20 to C21, C21 to C22, C22 to C23, C23 to C24, R29 to R30

Commit message: Update
Parts:
- renumbered C10 to C15, C11 to C16, C12 to C17, C13 to C18, C14 to C19, C15 to C20, C16 to C21, C17 to C22, C18 to C23, C19 to C24, C20 to C25, C21 to C26, C22 to C27, C23 to C28, C24 to C29, R30 to R40

Commit message: Update
Parts:
- removed C15: 1uF, symbol Device:C
- removed C20, C22: C, symbol Device:C
- removed C25, C26, C27: 100nF, symbol Device:C
- added C16: 20pF, symbol Device:C
- added C23: 100nF, symbol Device:C
- C17: value 100nF -> 20pF
- renumbered C18 to C15, C16 to C18, C21 to C20, C23 to C21, C24 to C22, C28 to C24, C29 to C25, R40 to R41
Connections:
- net +3V3: now also U9.1 (VBAT), U9.19 (VDD), U9.32 (VDD), U9.48 (VDD), U9.64 (VDD), C23.1
- net +3V3A: now also U9.13 (VDDA); no longer C17.1
- net BOOT0: now also U9.60 (PH3)
- net GND: now also U9.12 (VSSA), U9.18 (VSS), U9.31 (VSS), U9.47 (VSS), U9.63 (VSS), C16.2, C23.2
- net NRST: now also U9.7 (NRST)
- net at Y1.1: now also U9.5 (PH0), C16.1
- net at Y1.2: now also C17.1, U9.6 (PH1)
- net PC2: now reaches U9.10 (PC2)
- net PC3: now reaches U9.11 (PC3)
- net PA0: now reaches U9.14 (PA0)
- net PA1: now reaches U9.15 (PA1)
- net PA2: now reaches U9.16 (PA2)
- net PA3: now reaches U9.17 (PA3)
- net PC13: now reaches U9.2 (PC13)
- net PA4: now reaches U9.20 (PA4)
- net PA5: now reaches U9.21 (PA5)
- net PA6: now reaches U9.22 (PA6)
- net PA7: now reaches U9.23 (PA7)
- net PC4: now reaches U9.24 (PC4)
- net PC5: now reaches U9.25 (PC5)
- net PB0: now reaches U9.26 (PB0)
- net PB1: now reaches U9.27 (PB1)
- net PB2: now reaches U9.28 (PB2)
- net PB10: now reaches U9.29 (PB10)
- net PC14: now reaches U9.3 (PC14)
- net PB11: now reaches U9.30 (PB11)
- net PB12: now reaches U9.33 (PB12)
- net PB13: now reaches U9.34 (PB13)
- net PB14: now reaches U9.35 (PB14)
- net PB15: now reaches U9.36 (PB15)
- net PC6: now reaches U9.37 (PC6)
- net PC7: now reaches U9.38 (PC7)
- net PC8: now reaches U9.39 (PC8)
- net PC15: now reaches U9.4 (PC15)
- net PC9: now reaches U9.40 (PC9)
- net PA8: now reaches U9.41 (PA8)
- net PA9: now reaches U9.42 (PA9)
- net PA10: now reaches U9.43 (PA10)
- net PA11: now reaches U9.44 (PA11)
- net PA12: now reaches U9.45 (PA12)
- net PA13: now reaches U9.46 (PA13)
- net PA14: now reaches U9.49 (PA14)
- net PA15: now reaches U9.50 (PA15)
- net PC10: now reaches U9.51 (PC10)
- net PC11: now reaches U9.52 (PC11)
- net PC12: now reaches U9.53 (PC12)
- net PD2: now reaches U9.54 (PD2)
- net PB3: now reaches U9.55 (PB3)
- net PB4: now reaches U9.56 (PB4)
- net PB5: now reaches U9.57 (PB5)
- net PB6: now reaches U9.58 (PB6)
- net PB7: now reaches U9.59 (PB7)
- net PB8: now reaches U9.61 (PB8)
- net PB9: now reaches U9.62 (PB9)
- net PC0: now reaches U9.8 (PC0)
- net PC1: now reaches U9.9 (PC1)
Other:
- note added: "ADC1_IN5 (Potentiometer)"
- note added: "BQ24072_BATT_DISCHARGE"
- note added: "CAN1_RX (MCP2562)"
- note added: "CAN1_TX (MCP2562)"
- note added: "CAN_STBY (MCP2562)"
- note added: "ENABLE (7-Segment)"
- note added: "ENABLE (Buzzer)"
- note added: "ENABLE (LCD Backlight)"
- note added: "ENABLE (User LED)"
- note added: "I2C1_SCL (TMP1075)"
- note added: "I2C1_SDA (TMP1075)"
- note added: "I2C1_SMBA (TMP1075)"
- note added: "In-Application Programming (IAP): USART1 (PA9 and PA10) can be used for flashing new firmware to the MCU through ST's system bootloader or a custom one."
- note added: "LCD_D0"
- note added: "LCD_D1"
- note added: "LCD_D2"
- note added: "LCD_D3"
- note added: "LCD_D4"
- note added: "LCD_D5"
- note added: "LCD_D6"
- note added: "LCD_D7"
- note added: "LCD_ENABLE"
- note added: "LCD_RS"
- note added: "LIS3DH_INT1"
- note added: "LIS3DH_INT2"
- note added: "Microcontroller (MCU)"
- note added: "SEG_A (7-Segment)"
- note added: "SEG_B (7-Segment)"
- note added: "SEG_C (7-Segment)"
- note added: "SEG_D (7-Segment)"
- note added: "SEG_DP (7-Segment)"
- note added: "SEG_E (7-Segment)"
- note added: "SEG_F (7-Segment)"
- note added: "SEG_G (7-Segment)"
- note added: "SPI3_MISO (LIS3DH)"
- note added: "SPI3_MOSI (LIS3DH)"
- note added: "SPI3_SCK (LIS3DH)"
- note added: "SPI_CS (LIS3DH)"
- note added: "SWCLK (To ST-Link)"
- note added: "SWDIO (To ST-Link)"
- note added: "USART1_RX (For In-Application Programming)"
- note added: "USART1_TX (For In-Application Programming)"
- note added: "User Button"
- moved on the sheet: C15, C18, C19, C20, C21, C22, C24, C25, R41, SW3, U9, Y1
