File: rjx_training_kit/displays.kicad_sch (KiCad schematic)
At the start: 25 parts, among them Q1 BC847, Q2 BC857, Q3 BC857, Q4 BC857, Q5 BC857, Q6 BC857, U4 LTC-4627JD (Red)

Commit message: Update
Connections:
- net +3.3V renamed +3V3
Changed lines of the file:
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@@
 			)
 		)
-		(property "Value" "+3.3V"
+		(property "Value" "+3V3"
 			(at 153.67 85.09 0)
 			(effects
@@
 			)
 		)
-		(property "Value" "+3.3V"
+		(property "Value" "+3V3"
 			(at 153.67 46.99 0)
 			(effects
@@
 			)
 		)
-		(property "Value" "+3.3V"
+		(property "Value" "+3V3"
 			(at 153.67 123.19 0)
 			(effects
@@
 			)
 		)
-		(property "Value" "+3.3V"
+		(property "Value" "+3V3"
 			(at 153.67 104.14 0)
 			(effects
@@
 		(on_board yes)
 		(dnp no)
-		(fields_autoplaced yes)
 		(property "Reference" "#PWR016"
 			(at 68.58 88.9 0)
@@
 		)
 		(property "Value" "GND"
-			(at 68.58 87.63 0)
+			(at 68.58 86.614 0)
 			(effects
 				(font
@@
 			)
 		)
-		(property "Value" "+3.3V"
+		(property "Value" "+3V3"
 			(at 153.67 66.04 0)
 			(effects

Commit message: Update
Changed lines of the file:
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@@
 	(text "7 Segment Display"
 		(exclude_from_sim no)
-		(at 201.168 70.358 0)
+		(at 201.168 69.088 0)
 		(effects
 			(font
@@
 	(text "LCD"
 		(exclude_from_sim no)
-		(at 84.074 59.69 0)
+		(at 68.834 55.372 0)
 		(effects
 			(font

Commit message: Update
Parts:
- removed Q1: BC847, Package_TO_SOT_SMD:SOT-23, symbol Transistor_BJT:BC847
- removed Q2, Q3, Q4, Q5, Q6: BC857, Package_TO_SOT_SMD:SOT-23, symbol Transistor_BJT:BC857
- added Q1: BC817, Package_TO_SOT_SMD:SOT-23, symbol Transistor_BJT:BC817
- added Q2, Q3, Q4, Q5, Q6: BC808, Package_TO_SOT_SMD:SOT-23, symbol Transistor_BJT:BC808
- added R33, R34, R35, R36, R37: 10k, symbol Device:R_US
- R13, R14, R15, R16, R17: value 10k -> 510
- R7: value 10k -> 470
Connections:
- net +3V3: now also Q2.2 (E), Q3.2 (E), Q4.2 (E), Q5.2 (E), Q6.2 (E), R33.2, R34.2, R35.2, R36.2, R37.2
- net GND: now also Q1.2 (E)
- net PD11: now also R33.1
- net PD12: now also R34.1
- net PD13: now also R35.1
- net PD14: now also R36.1
- net PD15: now also R37.1
- net at R14.2: now also Q3.1 (B)
- net at U4.2 (CA2): now also Q3.3 (C)
- net at R7.2: now also Q1.1 (B)
- net at R17.2: now also Q6.1 (B)
- net at R16.2: now also Q5.1 (B)
- net at R15.2: now also Q4.1 (B)
- net at DS1.16 (LED(-)): now also Q1.3 (C)
- net at R13.2: now also Q2.1 (B)
- net at U4.1 (CA1): now also Q2.3 (C)
- net at U4.6 (CA3): now also Q4.3 (C)
- net at U4.4 (CAL): now also Q6.3 (C)
- net at U4.8 (CA4): now also Q5.3 (C)
Other:
- note added: ". PD11 to PD15 are floating inputs during and after a reset. . R33 to R37 pull these respective pins to 3.3V. . This keeps Q2 to Q6 off by default."
- note added: "Pull-Up Resistors"
- title: (none) -> Displays
- moved on the sheet: DS1, R13, R14, R15, R16, R17, R18, R19, R20, R21, R22, R23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

Commit message: Update
Connections:
- net B: now reaches R19.2, U4.16 (B)
- net CA2: now reaches Q3.3 (C), U4.2 (CA2)
- net C: now reaches R20.2, U4.13 (C)
- net CA4: now reaches Q5.3 (C), U4.8 (CA4)
- net F: now reaches R23.2, U4.11 (F)
- net CA3: now reaches Q4.3 (C), U4.6 (CA3)
- net G: now reaches R24.2, U4.15 (G)
- net CA1: now reaches Q2.3 (C), U4.1 (CA1)
- net DP: now reaches R25.2, U4.7 (DP)
- net D: now reaches R21.2, U4.3 (D)
- net E: now reaches R22.2, U4.5 (E)
- net CAL: now reaches Q6.3 (C), U4.4 (CAL)
- net A: now reaches R18.2, U4.14 (A)
Other:
- note added: "Cathodes"
- note added: "Common Anodes"
- moved on the sheet: DS1, Q1, Q2, Q3, Q4, Q5, Q6, R13, R14, R15, R16, R17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

Commit message: Update
Other:
- moved on the sheet: Q1, R6, R7, R8

Commit message: Update
Connections:
- net A: no longer names the net of R18.2, U4.14 (A)
- net B: no longer names the net of R19.2, U4.16 (B)
- net C: no longer names the net of R20.2, U4.13 (C)
- net CA1: no longer names the net of Q2.3 (C), U4.1 (CA1)
- net CA2: no longer names the net of Q3.3 (C), U4.2 (CA2)
- net CA3: no longer names the net of Q4.3 (C), U4.6 (CA3)
- net CA4: no longer names the net of Q5.3 (C), U4.8 (CA4)
- net CAL: no longer names the net of Q6.3 (C), U4.4 (CAL)
- net D: no longer names the net of R21.2, U4.3 (D)
- net DP: no longer names the net of R25.2, U4.7 (DP)
- net E: no longer names the net of R22.2, U4.5 (E)
- net F: no longer names the net of R23.2, U4.11 (F)
- net G: no longer names the net of R24.2, U4.15 (G)
Other:
- note removed: "Cathodes"
- note removed: "Common Anodes"
- moved on the sheet: DS1, Q1, Q2, Q3, Q4, Q5, Q6, R13, R14, R15, R16, R17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

Commit message: Update
Parts:
- R18: renamed from R7; value 470 -> 2k
- R25: renamed from R13; value 510 -> 2k
- R26: renamed from R14; value 510 -> 2k
- R27: renamed from R15; value 510 -> 2k
- R28: renamed from R16; value 510 -> 2k
- R29: renamed from R17; value 510 -> 2k
- R30: renamed from R18; value 240 -> 300
- R31: renamed from R19; value 240 -> 300
- R32: renamed from R20; value 240 -> 300
- R33: renamed from R21; value 240 -> 300
- R34: renamed from R22; value 240 -> 300
- R35: renamed from R23; value 240 -> 300
- R36: renamed from R24; value 240 -> 300
- R37: renamed from R25; value 240 -> 300
- renumbered Q1 to Q3, Q2 to Q4, Q3 to Q5, Q4 to Q6, Q5 to Q7, Q6 to Q8, R6 to R17, R8 to R19, R33 to R20, R34 to R21, R35 to R22, R36 to R23, R37 to R24, RV1 to RV2, U4 to U8
Other:
- note added: ". PD11 to PD15 are floating inputs during and after a reset. . R20 to R24 pull these respective pins to 3.3V. . This keeps Q4 to Q8 off by default."
- note removed: ". PD11 to PD15 are floating inputs during and after a reset. . R33 to R37 pull these respective pins to 3.3V. . This keeps Q2 to Q6 off by default."

Commit message: Update
Parts:
- R23: renamed from R19; value 240 -> 300
- renumbered R17 to R21, R18 to R22, R20 to R24, R21 to R25, R22 to R26, R23 to R27, R24 to R28, R25 to R29, R26 to R30, R27 to R31, R28 to R32, R29 to R33, R30 to R34, R31 to R35, R32 to R36, R33 to R37, R34 to R38, R35 to R39, R36 to R40, R37 to R41
Other:
- note removed: ". PD11 to PD15 are floating inputs during and after a reset. . R20 to R24 pull these respective pins to 3.3V. . This keeps Q4 to Q8 off by default."
