File: rjx_training_kit/displays.kicad_sch (KiCad schematic)
At the start: 30 parts, among them Q3 BC817, Q4 BC808, Q5 BC808, Q6 BC808, Q7 BC808, Q8 BC808, U8 LTC-4627JD (Red)

Commit message: Update
Parts:
- renumbered R21 to R24, R22 to R25, R23 to R26, R24 to R27, R25 to R28, R26 to R29, R27 to R30, R28 to R31, R29 to R32, R30 to R33, R31 to R34, R32 to R35, R33 to R36, R34 to R37, R35 to R38, R36 to R39, R37 to R40, R38 to R41, R39 to R42, R40 to R43, R41 to R44
Other:
- note added: "LCD Backlight ON/OFF Control"
- note added: "Note: These resistors pull PD11-15 to 3.3V because these pins float during and after a reset. This setup ensures transistors Q4 to Q8 have well-defined default states."

Commit message: Update
Parts:
- removed DS1: WC1602A, Display:WC1602A, symbol Display_Character:WC1602A
- removed Q3: BC817, Package_TO_SOT_SMD:SOT-23, symbol Transistor_BJT:BC817
- removed Q4, Q5, Q6, Q7, Q8: BC808, Package_TO_SOT_SMD:SOT-23, symbol Transistor_BJT:BC808
- removed R24, R27, R28, R29, R30, R31: 10k, symbol Device:R_US
- removed R25, R32, R33, R34, R35, R36: 2k, symbol Device:R_US
- removed R26, R37, R38, R39, R40, R41, R42, R43, R44: 300, symbol Device:R_US
- removed RV2: 10k, symbol Device:R_Potentiometer_Trim_US
- removed U8: LTC-4627JD (Red), Display_7Segment:LTC-4627Jx, symbol Display_Character:LTC-4627JD
Other:
- note removed: "7 Segment Display"
- note removed: "LCD"
- note removed: "LCD Backlight ON/OFF Control"
- note removed: "Note: These resistors pull PD11-15 to 3.3V because these pins float during and after a reset. This setup ensures transistors Q4 to Q8 have well-defined default states."
- note removed: "Pull-Up Resistors"
