File: rjx_training_kit/rjx_training_kit.kicad_sch (KiCad schematic)
At the start: 0 parts

Commit message: Update
Other:
- added sheet Displays (displays.kicad_sch)
- added sheet USB OTG (usb_otg.kicad_sch)
Changed lines of the file:
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@@
+	)
+	(sheet
+		(at 46.99 83.82)
+		(size 12.7 3.81)
+		(fields_autoplaced yes)
+		(stroke
+			(width 0.1524)
+			(type solid)
+		)
+		(fill
+			(color 0 0 0 0.0000)
+		)
+		(property "Sheetname" "USB OTG"
+			(at 46.99 83.1084 0)
+			(effects
+				(font
+					(size 1.27 1.27)
+				)
+				(justify left bottom)
+			)
+		)
+		(property "Sheetfile" "usb_otg.kicad_sch"
+			(at 46.99 88.2146 0)
+			(effects
+				(font
+					(size 1.27 1.27)
+				)
+				(justify left top)
+			)
+		)
+		(instances
+			(project "rjx_training_kit"
+				(path "/c10d0f5f-1570-4ced-80f8-bf69ea514c66"
+					(page "5")
+				)
+			)
+		)
 	)
 	(sheet
@@
 				)
 			)
+		)
+	)
+	(sheet
+		(at 69.85 110.49)
+		(size 12.7 3.81)
+		(fields_autoplaced yes)
+		(stroke
+			(width 0.1524)
+			(type solid)
+		)
+		(fill
+			(color 0 0 0 0.0000)
+		)
+		(property "Sheetname" "Displays"
+			(at 69.85 109.7784 0)
+			(effects
+				(font
+					(size 1.27 1.27)
+				)
+				(justify left bottom)
+			)
+		)
+		(property "Sheetfile" "displays.kicad_sch"
+			(at 69.85 114.8846 0)
+			(effects
+				(font
+					(size 1.27 1.27)
+				)
+				(justify left top)
+			)
+		)
+		(instances
+			(project "rjx_training_kit"
+				(path "/c10d0f5f-1570-4ced-80f8-bf69ea514c66"
+					(page "6")
+				)
+			)

Commit message: Update
Other:
- removed sheet USB OTG
- sheet Displays ports: added PB0, PB1, PB2, PB3, PB4, PB5, PB6, PB7, PD0, PD1, PD11, PD12, PD13, PD14, PD15, PD2, PD3, PD4, PD5, PD6, PD7, PE10, PE8, PE9; removed none
- sheet Microcontroller ports: added BOOT0, NRST, PA1, PA5, PA6, PA7, PB0, PB1, PB10, PB11, PB2, PB3, PB4, PB5, PB6, PB7, PC14, PC15, PC4, PC5, PD0, PD1, PD11, PD12, PD13, PD14, PD15, PD2, PD3, PD4, PD5, PD6, PD7, PE0, PE1, PE10, PE11, PE2, PE7, PE8, PE9, PH0, PH1; removed none
- sheet Peripherals ports: added PA1, PA5, PA6, PA7, PB10, PB11, PC4, PC5, PE0, PE1, PE11, PE2, PE7; removed none

Commit message: Update
Parts:
- added H1, H2, H3, H4: MountingHole, symbol Mechanical:MountingHole
Other:
- sheet Microcontroller ports: added PA0, PA10, PA11, PA12, PA13, PA14, PA15, PA2, PA3, PA4, PA8, PA9, PB12, PB13, PB14, PB15, PB8, PB9, PC0, PC1, PC10, PC11, PC12, PC13, PC2, PC3, PC6, PC7, PC8, PC9, PD10, PD8, PD9, PE12, PE13, PE14, PE15, PE3, PE4, PE5, PE6; removed none

Commit message: Update
Parts:
- added C1, C30: C_Polarized, symbol Device:C_Polarized
- added C2, C28, C29: C, symbol Device:C
- added D1: Power LED (Red), symbol Device:LED
- added J1: Barrel_Jack_Switch, symbol Connector:Barrel_Jack_Switch
- added L1: L, symbol Device:L
- added R1: 1.5k, symbol Device:R_US
- added R2, R3: R_US, symbol Device:R_US
- added SW1: SW_SPDT, symbol Switch:SW_SPDT
- added U6: TLV76133DCY, Package_TO_SOT_SMD:SOT-223-3_TabPin2, symbol Regulator_Linear:TLV76133DCY
- added U7: LM2596S-ADJ, Package_TO_SOT_SMD:TO-263-5_TabPin3, symbol Regulator_Switching:LM2596S-ADJ
Connections:
- new net: L1.2, U7.2 (OUT)
- new net: C29.1, R2.2, R3.1, U7.4 (FB)
- new net: J1.1, SW1.2 (B)
- new net: D1.2 (A), R1.2
- new net +3V3: C29.2, C30.1, L1.1, R3.2
- new net +3V3A: C28.1, U6.2 (VO)
- new net +5V: C1.1, C2.1, R1.1, SW1.1 (A), U6.3 (VI), U7.1 (VIN)
- new net GND: C1.2, C2.2, C28.2, C30.2, D1.1 (K), J1.2, J1.3, R2.1, U6.1 (GND), U7.3 (GND), U7.5 (~{ON}/OFF)
- no-connect marks 0 -> 1
Other:
- removed sheet Power section
- note added: "Analog Power Supply"
- note added: "Digital Power Supply"
- note added: "Power LED"
- moved on the sheet: H1, H2, H3, H4

Commit message: Update
Parts:
- added J2: Conn_02x03, symbol Connector_Generic:Conn_02x03_Odd_Even
- added J3: ST-Link, symbol Connector_Generic:Conn_01x03
- renumbered C2 to C1, C1 to C2, C28 to C3, C29 to C4, C30 to C5, U6 to U1, U7 to U2
Connections:
- net +3V3: now also J2.1 (Pin_1)
- net GND: now also J2.3 (Pin_3), J2.5 (Pin_5), J3.3 (Pin_3)
- net PB2: now also J2.6 (Pin_6)
- new net BOOT0: J2.2 (Pin_2)
- new net NRST: J2.4 (Pin_4)
- new net SWCLK: J3.2 (Pin_2)
- new net SWDIO: J3.1 (Pin_1)
Other:
- sheet Microcontroller ports: added none; removed PH0, PH1
- note added: "BOOT1"
- note added: "Free GPIO pins"
- note added: "Mounting Holes"
- note added: "Reset & Boot Pins"
- note added: "ST-Link"
- moved on the sheet: H1, H2, H3, H4

Commit message: Update
Parts:
- added R2: 2k, symbol Device:R_US
- C1: value C -> 1uF
- C3: value C -> 2.2uF
- R1: value 1.5k -> 2k
- renumbered R2 to R3, R3 to R4
Connections:
- net +5V: now also R2.1
- net at D1.2 (A), R1.2: now also R2.2
Other:
- sheet Peripherals ports: added PE12, PE13; removed none
- note added: "5V,2A"
- moved on the sheet: D1, J3, R1

Commit message: Update
Parts:
- removed C2, C5: C_Polarized, symbol Device:C_Polarized
- removed J3: ST-Link, symbol Connector_Generic:Conn_01x03
- removed L1: L, symbol Device:L
- removed U2: LM2596S-ADJ, Package_TO_SOT_SMD:TO-263-5_TabPin3, symbol Regulator_Switching:LM2596S-ADJ
- added C3: 10uF, symbol Device:C
- added J2: ST-Link, symbol Connector_Generic:Conn_01x03
- added J3: RTC_CLKO, symbol Connector_Generic:Conn_01x02
- added R5: 10k, symbol Device:R_US
- added U2: LD39200DPUR, LD39200:DFN-8-1EP_4x4mm_P0.8mm_EP2.3x3.24mm, symbol Regulator_LDO:LD39200DPUR
- C4: value C -> 10uF
- J4: renamed from J2; value Conn_02x03 -> Reset & BOOT
- R3: value R_US -> 56k
- R4: value R_US -> 10k
- renumbered C3 to C2
Connections:
- net +3V3: now also C4.1, R3.2, R5.1, U2.1 (OUT), U2.2 (OUT); no longer C4.2, R4.2
- net +5V: now also C3.1, U2.6 (EN), U2.7 (IN), U2.8 (IN)
- net GND: now also C4.2, R4.1, C3.2, J2.3 (Pin_3), J3.2 (Pin_2), U2.4 (GND), U2.9; no longer R3.1
- net SWCLK: now also J2.2 (Pin_2)
- net SWDIO: now also J2.1 (Pin_1)
- new net: R3.1, R4.2, U2.3 (ADJ/SENSE)
- new net PG: R5.2, U2.5 (PG)
- new net RTC_CLKO: J3.1 (Pin_1)
Other:
- sheet Peripherals ports: added RTC_CLKO; removed PE13
- note added: "3.3V,1A"
- note added: "3.3V,2A LDO"
- note added: "Connectors"
- note added: "Isink = Vout/R5 = 3.3V/10k = 330uA"
- note added: "Isink(max) = 6mA"
- note added: "LDO Filter Capacitors"
- note added: "LDO Output Status"
- note added: "Note: Strictly for analog components Recommended load current: 300mA"
- note added: "Note: The maximum input voltage is 5V The 5V powers the LDOs, Power LED, and LCD."
- note added: "Note: This LDO powers 3.3V digital devices Recommended load current: 1.2A Vout = Vadj(1 + R3/R4), Vadj = 0.5V LDO on: EN > 1.2V LDO off: EN < 0.5V PG(Power Good): Hi-Z when Vout > 0.92 * 3.3 Lo-Z when Vout < 0.80 * 3.3"
- note added: "PG monitors the quality of the LDO's output."
- note added: "PG's Isink < Isink(max)"
- note added: "Power Adapter & Switch"
- note added: "RTC Clock Output"
- note removed: "Free GPIO pins"
- moved on the sheet: C1, C2, D1, J1, J4, R1, R2, SW1, U1

Commit message: Update
Parts:
- added J?: LD39200, symbol Connector_Generic:Conn_01x02
Connections:
- net GND: now also J?.2 (Pin_2)
- net PG: now also J?.1 (Pin_1)
Other:
- note added: "CIN"
- note added: "COUT"
- note added: "LD39200 Power Good"
- note added: "LDO Capacitors"
- note added: "Microcontroller Pins, ST-Link, and Test Points"
- note added: "Note: Strictly for analog components Recommended max load current: 300mA"
- note added: "Note: This LDO powers 3.3V digital devices Recommended max load current: 1.2A Vout = Vadj(1 + R3/R4), Vadj = 0.5V LDO on: EN > 1.2V LDO off: EN < 0.5V PG(Power Good): Hi-Z when Vout > 0.92 * 3.3 Lo-Z when Vout < 0.80 * 3.3"
- note added: "PCF8563 RTC Clock Output"
- note added: "Test: Probe RTC_CLKO with an oscilloscope. Freq(RTC_CLKO) -> 32.768kHz"
- note added: "Test: V(PG) -> 3.3V when output is ok V(PG) -> 0.0V when output is not ok Measure V(PG) with a multimeter."
- note removed: "Connectors"
- note removed: "LDO Filter Capacitors"
- note removed: "Note: Strictly for analog components Recommended load current: 300mA"
- note removed: "Note: This LDO powers 3.3V digital devices Recommended load current: 1.2A Vout = Vadj(1 + R3/R4), Vadj = 0.5V LDO on: EN > 1.2V LDO off: EN < 0.5V PG(Power Good): Hi-Z when Vout > 0.92 * 3.3 Lo-Z when Vout < 0.80 * 3.3"
- note removed: "RTC Clock Output"
- moved on the sheet: J2, J3
