File: rjx_training_kit/rjx_training_kit.kicad_sch (KiCad schematic)
At the start: 22 parts, among them J1 Barrel_Jack_Switch, J2 ST-Link, J3 RTC_CLKO, J4 Reset & BOOT, SW1 SW_SPDT, U1 TLV76133DCY, U2 LD39200DPUR

Commit message: Update
Parts:
- removed J3: RTC_CLKO, symbol Connector_Generic:Conn_01x02
- removed J4: Reset & BOOT, symbol Connector_Generic:Conn_02x03_Odd_Even
- removed R2: 2k, symbol Device:R_US
- R1: value 2k -> 1k5
- gave numbers to parts that had none: 1
- renumbered R3 to R2, R4 to R3, R5 to R4
Other:
- removed sheet Displays
- sheet Microcontroller ports: added none; removed PA0, PA1, PA10, PA11, PA12, PA13, PA14, PA15, PA2, PA3, PA4, PA5, PA6, PA7, PA8, PA9, PB0, PB1, PB10, PB11, PB12, PB13, PB14, PB15, PB2, PB3, PB4, PB5, PB6, PB7, PB8, PB9, PC0, PC1, PC10, PC11, PC12, PC13, PC14, PC15, PC2, PC3, PC4, PC5, PC6, PC7, PC8, PC9, PD0, PD1, PD10, PD11, PD12, PD13, PD14, PD15, PD2, PD3, PD4, PD5, PD6, PD7, PD8, PD9, PE0, PE1, PE10, PE11, PE12, PE13, PE14, PE15, PE2, PE3, PE4, PE5, PE6, PE7, PE8, PE9
- sheet Peripherals ports: added none; removed PB10, PB11, PE12, RTC_CLKO
- note added: "Connectors"
- note removed: "BOOT1"
- note removed: "Microcontroller Pins, ST-Link, and Test Points"
- note removed: "PCF8563 RTC Clock Output"
- note removed: "Reset & Boot Pins"
- note removed: "Test: Probe RTC_CLKO with an oscilloscope. Freq(RTC_CLKO) -> 32.768kHz"
- moved on the sheet: R1

Commit message: Update
Parts:
- D1: value Power LED (Red) -> Red
- R1: value 1k5 -> 1.5k
Changed lines of the file:
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@@
 		(on_board yes)
 		(dnp no)
-		(property "Reference" "#PWR016"
+		(property "Reference" "#PWR028"
 			(at 137.16 35.56 0)
 			(effects
@@
 			(project "rjx_training_kit"
 				(path "/c10d0f5f-1570-4ced-80f8-bf69ea514c66"
-					(reference "#PWR016")
+					(reference "#PWR028")
 					(unit 1)
 				)
@@
 		(on_board yes)
 		(dnp no)
-		(property "Reference" "#PWR04"
+		(property "Reference" "#PWR016"
 			(at 35.56 153.67 0)
 			(effects
@@
 			(project "rjx_training_kit"
 				(path "/c10d0f5f-1570-4ced-80f8-bf69ea514c66"
-					(reference "#PWR04")
+					(reference "#PWR016")
 					(unit 1)
 				)
@@
 			)
 		)
-		(property "Value" "1k5"
+		(property "Value" "1.5k"
 			(at 34.29 97.79 0)
 			(effects
@@
 		(on_board yes)
 		(dnp no)
-		(property "Reference" "#PWR03"
+		(property "Reference" "#PWR015"
 			(at 35.56 55.88 0)
 			(effects
@@
 			(project "rjx_training_kit"
 				(path "/c10d0f5f-1570-4ced-80f8-bf69ea514c66"
-					(reference "#PWR03")
+					(reference "#PWR015")
 					(unit 1)
 				)
@@
 		(on_board yes)
 		(dnp no)
-		(property "Reference" "#PWR07"
+		(property "Reference" "#PWR019"
 			(at 60.96 40.64 0)
 			(effects
@@
 			(project "rjx_training_kit"
 				(path "/c10d0f5f-1570-4ced-80f8-bf69ea514c66"
-					(reference "#PWR07")
+					(reference "#PWR019")
 					(unit 1)
 				)
@@
 		(on_board yes)
 		(dnp no)
-		(property "Reference" "#PWR06"
+		(property "Reference" "#PWR018"
 			(at 53.34 40.64 0)
 			(effects
@@
 			(project "rjx_training_kit"
 				(path "/c10d0f5f-1570-4ced-80f8-bf69ea514c66"
-					(reference "#PWR06")
+					(reference "#PWR018")
 					(unit 1)
 				)
@@
 		(on_board yes)
 		(dnp no)
-		(property "Reference" "#PWR05"
+		(property "Reference" "#PWR017"
 			(at 35.56 189.23 0)
 			(effects
@@
 			(project "rjx_training_kit"
 				(path "/c10d0f5f-1570-4ced-80f8-bf69ea514c66"
-					(reference "#PWR05")
+					(reference "#PWR017")
 					(unit 1)
 				)
@@
 			)
 		)
-		(property "Value" "Power LED (Red)"
+		(property "Value" "Red"
 			(at 36.83 108.2674 90)
 			(effects
@@
 		(on_board yes)
 		(dnp no)
-		(property "Reference" "#PWR013"
+		(property "Reference" "#PWR025"
 			(at 118.11 36.83 0)
 			(effects
@@
 			(project "rjx_training_kit"
 				(path "/c10d0f5f-1570-4ced-80f8-bf69ea514c66"
-					(reference "#PWR013")
+					(reference "#PWR025")
 					(unit 1)
 				)
@@
 		(on_board yes)
 		(dnp no)
-		(property "Reference" "#PWR011"
+		(property "Reference" "#PWR023"
 			(at 100.33 96.52 0)
 			(effects
@@
 			(project "rjx_training_kit"
 				(path "/c10d0f5f-1570-4ced-80f8-bf69ea514c66"
-					(reference "#PWR011")
+					(reference "#PWR023")
 					(unit 1)
 				)
@@
 		(on_board yes)
 		(dnp no)
-		(property "Reference" "#PWR08"
+		(property "Reference" "#PWR020"
 			(at 64.77 40.64 0)
 			(effects
@@
 			(project "rjx_training_kit"
 				(path "/c10d0f5f-1570-4ced-80f8-bf69ea514c66"
-					(reference "#PWR08")
+					(reference "#PWR020")
 					(unit 1)
 				)
@@
 		(on_board yes)
 		(dnp no)
-		(property "Reference" "#PWR015"
+		(property "Reference" "#PWR027"
 			(at 129.54 62.23 0)
 			(effects
@@
 			(project "rjx_training_kit"
 				(path "/c10d0f5f-1570-4ced-80f8-bf69ea514c66"
-					(reference "#PWR015")
+					(reference "#PWR027")
 					(unit 1)
 				)
@@
 		(on_board yes)
 		(dnp no)
-		(property "Reference" "#PWR02"
+		(property "Reference" "#PWR014"
 			(at 33.02 116.84 0)
 			(effects
@@
 			(project "rjx_training_kit"
 				(path "/c10d0f5f-1570-4ced-80f8-bf69ea514c66"
-					(reference "#PWR02")
+					(reference "#PWR014")
 					(unit 1)
 				)
@@
 		(on_board yes)
 		(dnp no)
-		(property "Reference" "#PWR09"
+		(property "Reference" "#PWR021"
 			(at 64.77 96.52 0)
 			(effects
@@
 			(project "rjx_training_kit"
 				(path "/c10d0f5f-1570-4ced-80f8-bf69ea514c66"
-					(reference "#PWR09")
+					(reference "#PWR021")
 					(unit 1)
 				)
@@
 		(on_board yes)
 		(dnp no)
-		(property "Reference" "#PWR010"
+		(property "Reference" "#PWR022"
 			(at 82.55 115.57 0)
 			(effects
@@
 			(project "rjx_training_kit"
 				(path "/c10d0f5f-1570-4ced-80f8-bf69ea514c66"
-					(reference "#PWR010")
+					(reference "#PWR022")
 					(unit 1)
 				)
@@
 		(on_board yes)
 		(dnp no)
-		(property "Reference" "#PWR01"
+		(property "Reference" "#PWR013"
 			(at 33.02 93.98 0)
 			(effects
@@
 			(project "rjx_training_kit"
 				(path "/c10d0f5f-1570-4ced-80f8-bf69ea514c66"
-					(reference "#PWR01")
+					(reference "#PWR013")
 					(unit 1)
 				)
@@
 		(on_board yes)
 		(dnp no)
-		(property "Reference" "#PWR019"
+		(property "Reference" "#PWR031"
 			(at 148.59 48.26 0)
 			(effects
@@
 			(project "rjx_training_kit"
 				(path "/c10d0f5f-1570-4ced-80f8-bf69ea514c66"
-					(reference "#PWR019")
+					(reference "#PWR031")
 					(unit 1)
 				)
@@
 		(on_board yes)
 		(dnp no)
-		(property "Reference" "#PWR018"
+		(property "Reference" "#PWR030"
 			(at 148.59 35.56 0)
 			(effects
@@
 			(project "rjx_training_kit"
 				(path "/c10d0f5f-1570-4ced-80f8-bf69ea514c66"
-					(reference "#PWR018")
+					(reference "#PWR030")
 					(unit 1)
 				)
@@
 		(on_board yes)
 		(dnp no)
-		(property "Reference" "#PWR017"
+		(property "Reference" "#PWR029"
 			(at 137.16 48.26 0)
 			(effects
@@
 			(project "rjx_training_kit"
 				(path "/c10d0f5f-1570-4ced-80f8-bf69ea514c66"
-					(reference "#PWR017")
+					(reference "#PWR029")
 					(unit 1)
 				)
@@
 		(on_board yes)
 		(dnp no)
-		(property "Reference" "#PWR012"
+		(property "Reference" "#PWR024"
 			(at 114.3 60.96 0)
 			(effects
@@
 			(project "rjx_training_kit"
 				(path "/c10d0f5f-1570-4ced-80f8-bf69ea514c66"
-					(reference "#PWR012")
+					(reference "#PWR024")
 					(unit 1)
 				)
@@
 		(on_board yes)
 		(dnp no)
-		(property "Reference" "#PWR014"
+		(property "Reference" "#PWR026"
 			(at 121.92 60.96 0)
 			(effects
@@
 			(project "rjx_training_kit"
 				(path "/c10d0f5f-1570-4ced-80f8-bf69ea514c66"
-					(reference "#PWR014")
-					(unit 1)
-				)
+					(reference "#PWR026")
+					(unit 1)
+				)

Commit message: Update
Parts:
- removed J2: ST-Link, symbol Connector_Generic:Conn_01x03
- removed J3: LD39200, symbol Connector_Generic:Conn_01x02
- removed R4: 10k, symbol Device:R_US
- added J2, J3: Conn_01x32_Pin, symbol Connector:Conn_01x32_Pin
- added Q1: BC817, Package_TO_SOT_SMD:SOT-23, symbol Transistor_BJT:BC817
- added R1: 10k, symbol Device:R_US
- added R2: 1.5k, symbol Device:R_US
- U2: footprint LD39200:DFN-8-1EP_4x4mm_P0.8mm_EP2.3x3.24mm -> SON_0DPUR_STM
- renumbered H4 to H2, H2 to H3, H3 to H4, R1 to R3, R2 to R4, R3 to R5
Connections:
- net +3V3: now also J2.16 (Pin_16), J2.17 (Pin_17), J3.1 (Pin_1), J3.17 (Pin_17), J3.30 (Pin_30)
- net +3V3A: now also J2.29 (Pin_29)
- net +5V: now also R1.2
- net BOOT0: now also J2.12 (Pin_12)
- net GND: now also J2.15 (Pin_15), J2.28 (Pin_28), J3.18 (Pin_18), J3.2 (Pin_2), J3.31 (Pin_31), Q1.2 (E); no longer D1.1 (K)
- net NRST: now also J2.23 (Pin_23)
- net PA0: now also J2.30 (Pin_30)
- net PA1: now also J2.31 (Pin_31)
- net PA10: now also J3.6 (Pin_6)
- net PA11: now also J3.5 (Pin_5)
- net PA12: now also J3.4 (Pin_4)
- net PA15: now also J2.2 (Pin_2)
- net PA2: now also J2.32 (Pin_32)
- net PA3: now also J3.32 (Pin_32)
- net PA4: now also J3.29 (Pin_29)
- net PA5: now also J3.28 (Pin_28)
- net PA6: now also J3.27 (Pin_27)
- net PA7: now also J3.26 (Pin_26)
- net PA8: now also J3.8 (Pin_8)
- net PA9: now also J3.7 (Pin_7)
- net PB10: now also J3.20 (Pin_20)
- net PB11: now also J3.19 (Pin_19)
- net PB12: now also J3.16 (Pin_16)
- net PB13: now also J3.15 (Pin_15)
- net PB14: now also J3.14 (Pin_14)
- net PB15: now also J3.13 (Pin_13)
- net PB8: now also J2.13 (Pin_13)
- net PB9: now also J2.14 (Pin_14)
- net PC0: now also J2.24 (Pin_24)
- net PC1: now also J2.25 (Pin_25)
- net PC10: now also J2.3 (Pin_3)
- net PC11: now also J2.4 (Pin_4)
- net PC12: now also J2.5 (Pin_5)
- net PC13: now also J2.18 (Pin_18)
- net PC14: now also J2.19 (Pin_19)
- net PC15: now also J2.20 (Pin_20)
- net PC2: now also J2.26 (Pin_26)
- net PC3: now also J2.27 (Pin_27)
- net PC4: now also J3.25 (Pin_25)
- net PC5: now also J3.24 (Pin_24)
- net PC6: now also J3.12 (Pin_12)
- net PC7: now also J3.11 (Pin_11)
- net PC8: now also J3.10 (Pin_10)
- net PC9: now also J3.9 (Pin_9)
- net PG: now also R1.1, R2.1
- net SWCLK: now also J2.1 (Pin_1)
- net SWDIO: now also J3.3 (Pin_3)
- new net: Q1.1 (B), R2.2
- new net: D1.1 (K), Q1.3 (C)
- new net PB0: J3.23 (Pin_23)
- new net PB1: J3.22 (Pin_22)
- new net PB2: J3.21 (Pin_21)
- new net PB3: J2.7 (Pin_7)
- new net PB4: J2.8 (Pin_8)
- new net PB5: J2.9 (Pin_9)
- new net PB6: J2.10 (Pin_10)
- new net PB7: J2.11 (Pin_11)
- new net PD2: J2.6 (Pin_6)
- no-connect marks 1 -> 3
Other:
- sheet Microcontroller ports: added PA0, PA1, PA10, PA11, PA12, PA13, PA14, PA15, PA2, PA3, PA4, PA5, PA6, PA7, PA8, PA9, PB0, PB1, PB10, PB11, PB12, PB13, PB14, PB15, PB2, PB3, PB4, PB5, PB6, PB7, PB8, PB9, PC0, PC1, PC10, PC11, PC12, PC13, PC14, PC15, PC2, PC3, PC4, PC5, PC6, PC7, PC8, PC9, PD2; removed none
- sheet Peripherals ports: added PA0, PA11, PA12, PA3, PA4, PA8, PB0, PB1, PB12, PB13, PB14, PB15, PB2, PB3, PB4, PB5, PB6, PB7, PB8, PB9, PC0, PC1, PC10, PC11, PC12, PC13, PC2, PC3, PC6, PC7, PC8, PC9, PD2; removed PA6, PA7, PE0, PE1, PE11, PE2, PE7
- note added: "3.3V,2A"
- note added: "5V,2A Adapter"
- note added: "ADC1_IN5 (Potentiometer)"
- note added: "BQ24072_BATT_DISCHARGE"
- note added: "CAN1_RX (MCP2562)"
- note added: "CAN1_TX (MCP2562)"
- note added: "CAN_STBY (MCP2562)"
- note added: "ENABLE (7-Segment)"
- note added: "ENABLE (Buzzer)"
- note added: "ENABLE (LCD Backlight)"
- note added: "ENABLE (User LED)"
- note added: "For powering analog components. Recommended maximum load current without heatsink: 300mA."
- note added: "Headers"
- note added: "I2C1_SCL (TMP1075)"
- note added: "I2C1_SDA (TMP1075)"
- note added: "I2C1_SMBA (TMP1075)"
- note added: "In-Application Programming (IAP): USART1 (PA9 and PA10) can be used for flashing new firmware to the MCU through ST's system bootloader or a custom one."
- note added: "LCD_D0"
- note added: "LCD_D1"
- note added: "LCD_D2"
- note added: "LCD_D3"
- note added: "LCD_D4"
- note added: "LCD_D5"
- note added: "LCD_D6"
- note added: "LCD_D7"
- note added: "LCD_ENABLE"
- note added: "LCD_RS"
- note added: "LIS3DH_INT1"
- note added: "LIS3DH_INT2"
- note added: "Note: This LDO powers 3.3V digital devices Recommended max load current: 1.2A Vout = Vadj(1 + R3/R4), Vadj = 0.5V LDO on: EN > 1.2V LDO off: EN < 0.5V"
- note added: "Power Good"
- note added: "Power Good(PG) status Low: Vout < 0.8 * Vout(nom) Hi-Z: Vout > 0.92 * Vout(nom) Vout(nom) = 3.3V"
- note added: "SEG_A (7-Segment)"
- note added: "SEG_B (7-Segment)"
- note added: "SEG_C (7-Segment)"
- note added: "SEG_D (7-Segment)"
- note added: "SEG_DP (7-Segment)"
- note added: "SEG_E (7-Segment)"
- note added: "SEG_F (7-Segment)"
- note added: "SEG_G (7-Segment)"
- note added: "SPI3_MISO (LIS3DH)"
- note added: "SPI3_MOSI (LIS3DH)"
- note added: "SPI3_SCK (LIS3DH)"
- note added: "SPI_CS (LIS3DH)"
- note added: "USART1_RX (For In-Application Programming)"
- note added: "USART1_TX (For In-Application Programming)"
- note added: "User Button"
- note added: "VBAT"
- note added: "VDD"
- note added: "VDDA"
- note added: "VSS"
- note added: "VSSA"
- note removed: "3.3V,2A LDO"
- note removed: "5V,2A"
- note removed: "Connectors"
- note removed: "Isink = Vout/R5 = 3.3V/10k = 330uA"
- note removed: "Isink(max) = 6mA"
- note removed: "LD39200 Power Good"
- note removed: "LDO Capacitors"
- note removed: "LDO Output Status"
- note removed: "Note: Strictly for analog components Recommended max load current: 300mA"
- note removed: "Note: The maximum input voltage is 5V The 5V powers the LDOs, Power LED, and LCD."
- note removed: "Note: This LDO powers 3.3V digital devices Recommended max load current: 1.2A Vout = Vadj(1 + R3/R4), Vadj = 0.5V LDO on: EN > 1.2V LDO off: EN < 0.5V PG(Power Good): Hi-Z when Vout > 0.92 * 3.3 Lo-Z when Vout < 0.80 * 3.3"
- note removed: "PG monitors the quality of the LDO's output."
- note removed: "PG's Isink < Isink(max)"
- note removed: "Power Adapter & Switch"
- note removed: "ST-Link"
- note removed: "Test: V(PG) -> 3.3V when output is ok V(PG) -> 0.0V when output is not ok Measure V(PG) with a multimeter."
- moved on the sheet: C3, C4, D1, H1, H2, H3, H4, J1, R3, R4, R5, SW1
