File: rjx_training_kit/Hardware/microcontroller.kicad_sch (KiCad schematic)
At the start: 15 parts, among them SW3 SW_Push, U9 STM32L431RCTx, Y1 8MHz

Commit message: [RJX]: New project structure
Parts:
- renumbered SW3 to SW2
Other:
- note removed: "ADC1_IN5 (Potentiometer)"
- moved on the sheet: C15, C16, C17, C18, C19, C20, C21, C22, C23, C24, C25, R41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
