File: rjx_training_kit/Hardware/rjx_training_kit.kicad_sch (KiCad schematic)
At the start: 21 parts, among them J1 Barrel_Jack_Switch, J2 Conn_01x32_Pin, J3 Conn_01x32_Pin, Q1 BC817, SW1 SW_SPDT, U1 TLV76133DCY, U2 LD39200DPUR

Commit message: [RJX]: New project structure
Parts:
- removed SW1: SW_SPDT, symbol Switch:SW_SPDT
- U2: footprint SON_0DPUR_STM -> Package_DFN_QFN:DFN-8-1EP_4x4mm_P0.8mm_EP2.3x3.24mm
Connections:
- net +5V: now also J1.1
- no-connect marks 3 -> 2
Other:
- sheet Peripherals ports: added none; removed PA0
- note removed: "ADC1_IN5 (Potentiometer)"
- moved on the sheet: J1
