File: rjx_training_kit/Hardware/rjx_training_kit.kicad_pcb (KiCad board)
At the start: 2 copper layers, 0 parts

Commit message: [RJX]: Schematic, Netlist, and PCB update. Replaced 2-pin crystal with 4-pin passive crystal.
Parts:
- added BZ1: 5V_Buzzer, Buzzer_Beeper:Buzzer_12x9.5RM7.6, F.Cu at (121.1, 88.4)
- added C1: 1uF, Capacitor_SMD:C_0603_1608Metric, F.Cu at (84.0, 49.5)
- added C10: 10uF, Capacitor_SMD:C_0603_1608Metric, F.Cu at (100.1, 69.2)
- added C11: 0.47uF, Capacitor_SMD:C_0603_1608Metric, F.Cu at (100.1, 71.7)
- added C12: 100nF, Capacitor_SMD:C_0603_1608Metric, F.Cu at (100.1, 74.2)
- added C13: 100nF, Capacitor_SMD:C_0603_1608Metric, F.Cu at (100.1, 76.7)
- added C14: 100nF, Capacitor_SMD:C_0603_1608Metric, F.Cu at (104.1, 56.6)
- added C15: 100nF, Capacitor_SMD:C_0603_1608Metric, F.Cu at (95.5, 112.9)
- added C16: 10pF, Capacitor_SMD:C_0603_1608Metric, F.Cu at (95.5, 115.4)
- added C17: 10pF, Capacitor_SMD:C_0603_1608Metric, F.Cu at (95.5, 117.9)
- added C18: 4.7uF, Capacitor_SMD:C_0603_1608Metric, F.Cu at (95.5, 120.4)
- added C19: 100nF, Capacitor_SMD:C_0603_1608Metric, F.Cu at (99.5, 112.9)
- added C2: 2.2uF, Capacitor_SMD:C_0603_1608Metric, F.Cu at (84.0, 52.0)
- added C20: 100nF, Capacitor_SMD:C_0603_1608Metric, F.Cu at (99.5, 115.4)
- added C21: 100nF, Capacitor_SMD:C_0603_1608Metric, F.Cu at (99.5, 117.9)
- added C22: 100nF, Capacitor_SMD:C_0603_1608Metric, F.Cu at (99.5, 120.4)
- added C23: 100nF, Capacitor_SMD:C_0603_1608Metric, F.Cu at (103.5, 112.9)
- added C24: 100nF, Capacitor_SMD:C_0603_1608Metric, F.Cu at (103.5, 115.4)
- added C25: 1uF, Capacitor_SMD:C_0603_1608Metric, F.Cu at (103.5, 117.9)
- added C3: 10uF, Capacitor_SMD:C_0603_1608Metric, F.Cu at (84.0, 54.5)
- added C4: 10uF, Capacitor_SMD:C_0603_1608Metric, F.Cu at (84.0, 57.0)
- added C5: 1uF, Capacitor_SMD:C_0603_1608Metric, F.Cu at (100.1, 56.6)
- added C6: 1uF, Capacitor_SMD:C_0603_1608Metric, F.Cu at (100.1, 59.1)
- added C7: 4.7uF, Capacitor_SMD:C_0603_1608Metric, F.Cu at (100.1, 61.7)
- added C8: 4.7uF, Capacitor_SMD:C_0603_1608Metric, F.Cu at (100.1, 64.2)
- added C9: 100nF, Capacitor_SMD:C_0603_1608Metric, F.Cu at (100.1, 66.7)
- added D1: Red, LED_SMD:LED_0603_1608Metric, F.Cu at (81.4, 100.7)
- added D2: Green, LED_SMD:LED_0603_1608Metric, F.Cu at (110.7, 79.3)
- added D3: Yellow, LED_SMD:LED_0603_1608Metric, F.Cu at (110.7, 81.9)
- added D4: Orange, LED_SMD:LED_0603_1608Metric, F.Cu at (110.7, 84.5)
- added D5: Green, LED_SMD:LED_0603_1608Metric, F.Cu at (110.7, 87.0)
- added DS1: WC1602A, Connector_PinSocket_2.54mm:PinSocket_1x16_P2.54mm_Vertical, F.Cu at (95.8, 50.6)
- added H1: MountingHole, MountingHole:MountingHole_3mm, F.Cu at (78.2, 52.0)
- added H2: MountingHole, MountingHole:MountingHole_3mm, F.Cu at (78.2, 59.6)
- added H3: MountingHole, MountingHole:MountingHole_3mm, F.Cu at (78.2, 67.1)
- added H4: MountingHole, MountingHole:MountingHole_3mm, F.Cu at (78.2, 74.7)
- added J1: Barrel_Jack_Switch, Connector_BarrelJack:BarrelJack_Horizontal, F.Cu at (89.0, 83.8)
- added J2: Conn_01x32_Pin, Connector_PinHeader_2.54mm:PinHeader_1x32_P2.54mm_Vertical, F.Cu at (67.5, 50.5)
- added J3: Conn_01x32_Pin, Connector_PinHeader_2.54mm:PinHeader_1x32_P2.54mm_Vertical, F.Cu at (72.1, 50.5)
- added J4: LiPo_4.2V, Connector_JST:JST_PH_S2B-PH-K_1x02_P2.00mm_Horizontal, F.Cu at (126.0, 57.8)
- added J5: LiPo_4.2V, Connector_JST:JST_PH_S2B-PH-K_1x02_P2.00mm_Horizontal, F.Cu at (134.0, 57.8)
- added J6: CHG_OUT, Connector_PinHeader_2.54mm:PinHeader_1x02_P2.54mm_Vertical, F.Cu at (100.4, 50.5)
- added J7: CAN_Bus, Connector_PinHeader_2.54mm:PinHeader_1x02_P2.54mm_Vertical, F.Cu at (105.0, 50.5)
- added J8: CAN_Bus, Connector_PinHeader_2.54mm:PinHeader_1x02_P2.54mm_Vertical, F.Cu at (109.6, 50.5)
- added JP1: Jumper_2_Open, Connector_PinHeader_2.54mm:PinHeader_1x02_P2.54mm_Vertical, F.Cu at (114.1, 50.5)
- added JP2: Jumper_2_Open, Connector_PinHeader_2.54mm:PinHeader_1x02_P2.54mm_Vertical, F.Cu at (118.7, 50.5)
- added JP3: Jumper_2_Open, Connector_PinHeader_2.54mm:PinHeader_1x02_P2.54mm_Vertical, F.Cu at (123.3, 50.5)
- added JP4: Jumper_2_Open, Connector_PinHeader_2.54mm:PinHeader_1x02_P2.54mm_Vertical, F.Cu at (127.9, 50.5)
- added Q1: BC817, Package_TO_SOT_SMD:SOT-23, F.Cu at (76.9, 101.6)
- added Q2: BC817, Package_TO_SOT_SMD:SOT-23, F.Cu at (120.6, 57.6)
- added Q3: BC817, Package_TO_SOT_SMD:SOT-23, F.Cu at (120.6, 62.1)
- added Q4: BC808, Package_TO_SOT_SMD:SOT-23, F.Cu at (120.6, 66.5)
- added Q5: BC817, Package_TO_SOT_SMD:SOT-23, F.Cu at (120.6, 71.0)
- added R1: 10k, Resistor_SMD:R_0603_1608Metric, F.Cu at (84.0, 59.5)
- added R10: 1.8M, Resistor_SMD:R_0603_1608Metric, F.Cu at (104.1, 69.2)
- added R11: 10k, Resistor_SMD:R_0603_1608Metric, F.Cu at (104.1, 71.7)
- added R12: 10k, Resistor_SMD:R_0603_1608Metric, F.Cu at (104.1, 74.2)
- added R13: 10m, Resistor_SMD:R_2512_6332Metric, F.Cu at (136.0, 84.1)
- added R14: 300, Resistor_SMD:R_0603_1608Metric, F.Cu at (104.1, 76.7)
- added R15: 1.5k, Resistor_SMD:R_0603_1608Metric, F.Cu at (108.1, 56.6)
- added R16: 1.5k, Resistor_SMD:R_0603_1608Metric, F.Cu at (108.1, 59.1)
- added R17: 300, Resistor_SMD:R_0603_1608Metric, F.Cu at (108.1, 61.7)
- added R18: 33, Resistor_SMD:R_2512_6332Metric, F.Cu at (136.0, 89.0)
- added R19: 300, Resistor_SMD:R_0603_1608Metric, F.Cu at (108.1, 64.2)
- added R2: 1.5k, Resistor_SMD:R_0603_1608Metric, F.Cu at (84.0, 62.0)
- added R20: 4.7k, Resistor_SMD:R_0603_1608Metric, F.Cu at (108.1, 66.7)
- added R21: 300, Resistor_SMD:R_0603_1608Metric, F.Cu at (108.1, 69.2)
- added R22: 300, Resistor_SMD:R_0603_1608Metric, F.Cu at (108.1, 71.7)
- added R23: 300, Resistor_SMD:R_0603_1608Metric, F.Cu at (108.1, 74.2)
- added R24: 300, Resistor_SMD:R_0603_1608Metric, F.Cu at (108.1, 76.7)
- added R25: 300, Resistor_SMD:R_0603_1608Metric, F.Cu at (112.1, 56.6)
- added R26: 300, Resistor_SMD:R_0603_1608Metric, F.Cu at (112.1, 59.1)
- added R27: 300, Resistor_SMD:R_0603_1608Metric, F.Cu at (112.1, 61.7)
- added R28: 300, Resistor_SMD:R_0603_1608Metric, F.Cu at (112.1, 64.2)
- added R29: 10k, Resistor_SMD:R_0603_1608Metric, F.Cu at (112.1, 66.7)
- added R3: 1.5k, Resistor_SMD:R_0603_1608Metric, F.Cu at (84.0, 64.6)
- added R30: 1.5k, Resistor_SMD:R_0603_1608Metric, F.Cu at (112.1, 69.2)
- added R31: 10k, Resistor_SMD:R_0603_1608Metric, F.Cu at (112.1, 71.7)
- added R32: 1.5k, Resistor_SMD:R_0603_1608Metric, F.Cu at (112.1, 74.2)
- added R33: 1.5k, Resistor_SMD:R_0603_1608Metric, F.Cu at (112.1, 76.7)
- added R34: 10k, Resistor_SMD:R_0603_1608Metric, F.Cu at (116.1, 56.6)
- added R35: 1.5k, Resistor_SMD:R_0603_1608Metric, F.Cu at (116.1, 59.1)
- added R36: 120, Resistor_SMD:R_0603_1608Metric, F.Cu at (116.1, 61.7)
- added R37: 300, Resistor_SMD:R_0603_1608Metric, F.Cu at (116.1, 64.2)
- added R38: 4.7k, Resistor_SMD:R_0603_1608Metric, F.Cu at (116.1, 66.7)
- added R39: 4.7k, Resistor_SMD:R_0603_1608Metric, F.Cu at (116.1, 69.2)
- added R4: 56k, Resistor_SMD:R_0603_1608Metric, F.Cu at (84.0, 67.1)
- added R40: 4.7k, Resistor_SMD:R_0603_1608Metric, F.Cu at (116.1, 71.7)
- added R41: 10k, Resistor_SMD:R_0603_1608Metric, F.Cu at (103.5, 120.4)
- added R5: 10k, Resistor_SMD:R_0603_1608Metric, F.Cu at (84.0, 69.6)
- added R6: 56k, Resistor_SMD:R_0603_1608Metric, F.Cu at (104.1, 59.1)
- added R7: 1.5k, Resistor_SMD:R_0603_1608Metric, F.Cu at (104.1, 61.7)
- added R8: 1.5k, Resistor_SMD:R_0603_1608Metric, F.Cu at (104.1, 64.2)
- added R9: 1.5k, Resistor_SMD:R_0603_1608Metric, F.Cu at (104.1, 66.7)
- added RV1: 10k, Potentiometer_THT:Potentiometer_Bourns_3296W_Vertical, F.Cu at (131.1, 68.2)
- added SW1: SW_Push, Button_Switch_THT:SW_PUSH_6mm, F.Cu at (100.1, 80.0)
- added SW2: SW_Push, Button_Switch_THT:SW_PUSH_6mm, F.Cu at (107.5, 113.7)
- added U1: TLV76133DCY, Package_TO_SOT_SMD:SOT-223-3_TabPin2, F.Cu at (79.4, 95.3)
- added U2: LD39200DPUR, Package_DFN_QFN:DFN-8-1EP_4x4mm_P0.8mm_EP2.3x3.24mm, F.Cu at (87.8, 93.8)
- added U3: BQ24072RGT, Package_DFN_QFN:VQFN-16-1EP_3x3mm_P0.5mm_EP1.6x1.6mm, F.Cu at (135.5, 75.8)
- added U4: LIS3DH, Package_LGA:LGA-16_3x3mm_P0.5mm_LayoutBorder3x5y, F.Cu at (115.3, 80.2)
- added U5: BQ27441-G1, Package_SON:Texas_S-PDSO-N12, F.Cu at (137.2, 67.3)
- added U6: KCSA02-136, Display_7Segment:KCSC02-136, F.Cu at (125.3, 77.4)
- added U7: TMP1075DGK, Package_SO:VSSOP-8_3x3mm_P0.65mm, F.Cu at (101.8, 88.9)
- added U8: MCP2562-E-SN, Package_SO:SOIC-8_3.9x4.9mm_P1.27mm, F.Cu at (112.9, 91.7)
- added U9: STM32L431RCTx, Package_QFP:LQFP-64_10x10mm_P0.5mm, F.Cu at (100.7, 104.4)
- added Y1: 8MHz, Crystal:Crystal_SMD_3225-4Pin_3.2x2.5mm, F.Cu at (110.6, 99.5)
